File: Dash.kicad_sch (KiCad schematic)
At the start: 13 parts, among them U1 ESP32-S2-DevKitM, U2 PCA9685PW

Commit message: Uploaded correct versions
uploading correct versions of schematics
Parts:
- removed R1, R2: 10K, symbol Device:R
- added C1, C2: C_Polarized, symbol Device:C_Polarized
- added C10, C11, C12, C3, C4, C5: 15uF, symbol Device:C_Polarized
- added C13, C6: 0.47uF, symbol Device:C
- added C14, C7: 0.01uF, symbol Device:C
- added C15, C16, C8, C9: 180uF, symbol Device:C_Polarized
- added D5, D6: D_Schottky, symbol Device:D_Schottky
- added L1, L2: 22uH, symbol Device:L
- added Q1, Q2: 2N7000, Package_TO_SOT_THT:TO-92_Inline, symbol Transistor_FET:2N7000
- added R10, R11, R12, R13, R14, R15, R16, R35, R36, R37, R38, R8, R9: 220, symbol Device:R
- added R17, R18, R19, R20, R21, R22, R23, R24, R25, R26, R27, R28, R29, R30, R31, R32, R33, R34, R39, R6, R7: 10K, symbol Device:R
- added U3: LM2678T-3.3, symbol Buck-Converter:LM2678T-3.3
- added U4: LM2678T-5.0, symbol Buck-Converter:LM2678T-5.0
- added U5: PCA9685PW, Package_SO:TSSOP-28_4.4x9.7mm_P0.65mm, symbol Driver_LED:PCA9685PW
- added U6, U7: 24C02Cx-x-SN, Package_SO:SOIC-8_3.9x4.9mm_P1.27mm, symbol Memory_EEPROM:24C02Cx-x-SN
- renumbered D3 to D2, D2 to D3, R7 to R1, R6 to R2, U2 to U1, U1 to U2
Connections:
- net +3.3V: now also R3.1, U1.2 (A1), C1.1, C2.1, C8.1, C9.1, L1.2, Q1.2 (G), Q2.2 (G), R19.2, R20.2, R24.1, R26.1, U3.6 (Feedback), U5.1 (A0), U5.2 (A1), U5.28 (VDD)
- net GND: now also R1.1, R2.1, R4.1, R5.1, C1.2, C10.2, C11.2, C12.2, C13.2, C15.2, C16.2, C2.2, C3.2, C4.2, C5.2, C6.2, C8.2, C9.2, D5.2 (A), D6.2 (A), R18.1, R19.1, R20.1, R21.1, R22.1, R23.1, R28.1, R29.1, R30.1, R31.1, R32.1, R33.1, R34.1, R6.1, R7.1, U3.4 (GND), U4.4 (GND), U5.14 (VSS), U5.25 (EXTCLK), U6.4 (GND), U6.7 (WP), U7.4 (GND), U7.7 (WP); no longer R1.2, R2.2, R4.2, R5.2
- net Servo 1: now also R8.2; no longer U1.6 (LED0)
- net Servo 2: now also R9.2; no longer U1.7 (LED1)
- net Servo 3: now also R10.2; no longer U1.8 (LED2)
- net Servo 4: now also R11.2; no longer U1.9 (LED3)
- net Servo 5: now also R12.2; no longer U1.10 (LED4)
- net Servo 6: now also R13.2; no longer U1.11 (LED5)
- net at U1.4 (A3): now also R5.2; no longer R3.1
- net at U1.5 (A4): now also R6.2
- net at U1.1 (A0): now also R2.2; no longer R2.1
- net at U1.23 (~{OE}): now also R1.2; no longer R1.1
- net Temp LED: now reaches D2.4 (DI)
- net Temp LED: now also R36.2
- net at U1.24 (A5): now also R7.2
- net SCL: now reaches U1.26 (SCL)
- net SCL: now also U2.28 (GPIO34), U5.26 (SCL), U6.6 (SCL), U7.6 (SCL)
- net SDA: now reaches U1.27 (SDA)
- net SDA: now also U2.27 (GPIO33), R17.2, R39.2, U5.27 (SDA), U6.5 (SDA), U7.5 (SDA)
- net at U1.3 (A2): now also R4.2; no longer R4.1
- net Headlights On Off: now reaches U2.10 (GPIO8/TOUCH8/ADC1_CH7)
- net Ignition Sensor: now reaches U2.11 (GPIO9/TOUCH9/ADC1_CH8/FSPIHD)
- net Power Off: now reaches U2.12 (GPIO10/TOUCH10/ADC1_CH9/FSPICS0/FSPIIO4)
- net Tach In: now reaches U2.3 (GPIO1/TOUCH1/ADC1_CH0)
- net Speed In: now reaches U2.4 (GPIO2/TOUCH2/ADC1_CH1)
- net Temp In: now reaches U2.5 (GPIO3/TOUCH3/ADC1_CH2)
- net Batt In: now reaches U2.6 (GPIO4/TOUCH4/ADC1_CH3)
- net Fuel In: now reaches U2.7 (GPIO5/TOUCH5/ADC1_CH4)
- net Oil In: now reaches U2.8 (GPIO6/TOUCH6/ADC1_CH5)
- net Trip Reset: now reaches U2.9 (GPIO7/TOUCH7/ADC1_CH6)
- net Oil LED: now reaches D1.4 (DI)
- net Batt LED: now reaches D4.4 (DI)
- net Batt LED: now also R38.2
- net Fuel LED: now reaches D3.4 (DI)
- net Fuel LED: now also R37.2
- new net: R16.1, U5.12 (LED6)
- new net: R14.1, U5.10 (LED4)
- new net: R8.1, U1.6 (LED0)
- new net: R12.1, U1.10 (LED4)
- new net: R15.1, U5.11 (LED5)
- new net: R18.2, U5.23 (~{OE})
- new net: R28.2, U5.24 (A5)
- new net: R21.2, U5.3 (A2)
- new net: R22.2, U5.4 (A3)
- new net: R23.2, U5.5 (A4)
- new net: R35.1, U5.6 (LED0)
- new net: R36.1, U5.7 (LED1)
- new net: R37.1, U5.8 (LED2)
- new net: R38.1, U5.9 (LED3)
- new net: C7.1, U3.3 (CB)
- new net: C7.2, D5.1 (K), L1.1, U3.1 (Vout)
- new net: R9.1, U1.7 (LED1)
- new net: R33.2, U7.2 (A1)
- new net: C14.2, D6.1 (K), L2.1, U4.1 (Vout)
- new net: R34.2, U7.3 (A2)
- new net: R10.1, U1.8 (LED2)
- new net: C14.1, U4.3 (CB)
- new net: R13.1, U1.11 (LED5)
- new net: R11.1, U1.9 (LED3)
- new net: R29.2, U6.1 (A0)
- new net: R30.2, U6.2 (A1)
- new net: R31.2, U6.3 (A2)
- new net +5V: C15.1, C16.1, L2.2, R17.1, R25.1, R27.1, R32.2, R39.1, U4.6 (Feedback), U6.8 (VCC), U7.1 (A0), U7.8 (VCC)
- new net +BATT: C10.1, C11.1, C12.1, C13.1, C3.1, C4.1, C5.1, C6.1, U3.2 (Vin), U4.2 (Vin)
- new net LCD B Backlight: R16.2
- new net LCD G Backlight: R15.2
- new net LCD R Backlight: R14.2
- new net OIl LED: R35.2
- new net Signal In: Q1.3 (D), Q2.3 (D), R25.2, R27.2
- new net Signal Out: Q1.1 (S), Q2.1 (S), R24.2, R26.2
- no-connect marks 3 -> 15
Other:
- moved on the sheet: D1, D2, D3, D4, R1, R2

Commit message: added components
added power flags, servo connectors, optocoupler, and mosfet
Parts:
- removed U2: ESP32-S2-DevKitM, Espressif:ESP32-S2-DevKitM, symbol Espressif:ESP32-S2-DevKitM
- removed U3: LM2678T-3.3, symbol Buck-Converter:LM2678T-3.3
- removed U4: LM2678T-5.0, symbol Buck-Converter:LM2678T-5.0
- added J1, J2, J3, J4, J5, J6: Conn_01x03_Socket, symbol Connector:Conn_01x03_Socket
- added Q3: 2N7000, Package_TO_SOT_THT:TO-92_Inline, symbol Transistor_FET:2N7000
- added R40: 150, symbol Device:R
- added U2: LM2678T-3.3, symbol Buck-Converter:LM2678T-3.3
- added U3: LM2678T-5.0, symbol Buck-Converter:LM2678T-5.0
- added U8: SFH617A-1, Package_DIP:DIP-4_W7.62mm, symbol Isolator:SFH617A-1
- added U9: ESP32-S2-DevKitM, PCM_Espressif:ESP32-S2-DevKitM, symbol Espressif:ESP32-S2-DevKitM
Connections:
- net OIl LED is gone; now on net Oil LED: R35.2
- net +3.3V: now also U2.6 (Feedback), U8.4, U9.1 (3V3)
- net +5V: now also D1.3 (VDD), D2.3 (VDD), D3.3 (VDD), D4.3 (VDD), J1.2 (Pin_2), J2.2 (Pin_2), J3.2 (Pin_2), J4.2 (Pin_2), J5.2 (Pin_2), J6.2 (Pin_2), U3.6 (Feedback)
- net +BATT: now also U2.2 (Vin), U3.2 (Vin), U8.1
- net Batt In: now also U9.6 (GPIO4/TOUCH4/ADC1_CH3)
- net Fuel In: now also U9.7 (GPIO5/TOUCH5/ADC1_CH4)
- net GND: now also D1.2 (GND), D2.2 (GND), D3.2 (GND), D4.2 (GND), J1.1 (Pin_1), J2.1 (Pin_1), J3.1 (Pin_1), J4.1 (Pin_1), J5.1 (Pin_1), J6.1 (Pin_1), Q3.1 (S), R40.2, U2.4 (GND), U3.4 (GND), U9.21 (GND), U9.42 (GND)
- net Headlights On Off: now also U9.10 (GPIO8/TOUCH8/ADC1_CH7)
- net Ignition Sensor: now also U8.3, U9.11 (GPIO9/TOUCH9/ADC1_CH8/FSPIHD)
- net Oil In: now also U9.8 (GPIO6/TOUCH6/ADC1_CH5)
- net Power Off: now also Q3.2 (G), U9.12 (GPIO10/TOUCH10/ADC1_CH9/FSPICS0/FSPIIO4)
- net SCL: now also U9.28 (GPIO34)
- net SDA: now also U9.27 (GPIO33)
- net Servo 1: now also J1.3 (Pin_3)
- net Servo 2: now also J2.3 (Pin_3)
- net Servo 3: now also J3.3 (Pin_3)
- net Servo 4: now also J4.3 (Pin_3)
- net Servo 5: now also J5.3 (Pin_3)
- net Servo 6: now also J6.3 (Pin_3)
- net Speed In: now also U9.4 (GPIO2/TOUCH2/ADC1_CH1)
- net Tach In: now also U9.3 (GPIO1/TOUCH1/ADC1_CH0)
- net Temp In: now also U9.5 (GPIO3/TOUCH3/ADC1_CH2)
- net Trip Reset: now also U9.9 (GPIO7/TOUCH7/ADC1_CH6)
- net at C7.1: now also U2.3 (CB)
- net at C7.2, D5.1 (K), L1.1: now also U2.1 (Vout)
- net at C14.2, D6.1 (K), L2.1: now also U3.1 (Vout)
- net at C14.1: now also U3.3 (CB)
- new net: R40.1, U8.2
- new net +VDC: Q3.3 (D)
- no-connect marks 15 -> 19
Other:
- moved on the sheet: D1, D2, D3, D4

Commit message: Removed PCA chips
removed pca chips, added additional parts, moved leds to single bus
Parts:
- removed C1, C2: C_Polarized, symbol Device:C_Polarized
- removed R14, R15, R16, R35, R36, R37, R38: 220, symbol Device:R
- removed R18, R19, R2, R20, R21, R22, R23, R28, R3, R4, R5, R6, R7: 10K, symbol Device:R
- removed U1, U5: PCA9685PW, Package_SO:TSSOP-28_4.4x9.7mm_P0.65mm, symbol Driver_LED:PCA9685PW
- added D10, D11, D7, D8, D9: APA-106-F5, LED_THT:LED_D5.0mm-4_RGB, symbol LED:APA-106-F5
- added J7: Conn_01x04_Socket, symbol Connector:Conn_01x04_Socket
- added J8: Conn_01x07_Socket, symbol Connector:Conn_01x07_Socket
- added J9: Conn_01x06_Socket, symbol Connector:Conn_01x06_Socket
- added LS1: Speaker, symbol Device:Speaker
- added SW1: SW_Push, symbol Switch:SW_Push
Connections:
- net Batt LED is gone; now on an unnamed net: D4.4 (DI)
- net Fuel LED is gone; now on an unnamed net: D3.4 (DI)
- net Oil LED is gone; now on net LED Data Out: D1.4 (DI)
- net +3.3V: now also SW1.1
- net +5V: now also D10.3 (VDD), D11.3 (VDD), D7.3 (VDD), D8.3 (VDD), D9.3 (VDD), J7.4 (Pin_4), J8.2 (Pin_2)
- net Batt In: now also J9.3 (Pin_3)
- net Fuel In: now also J9.2 (Pin_2)
- net GND: now also R1.2, D10.2 (GND), D11.2 (GND), D7.2 (GND), D8.2 (GND), D9.2 (GND), J7.1 (Pin_1), J8.1 (Pin_1); no longer R1.1
- net Oil In: now also J9.1 (Pin_1)
- net Speed In: now also Q1.3 (D), R25.2, J9.6 (Pin_6); no longer U9.4 (GPIO2/TOUCH2/ADC1_CH1)
- net Tach In: now also Q2.3 (D), R27.2, J9.5 (Pin_5); no longer U9.3 (GPIO1/TOUCH1/ADC1_CH0)
- net Temp In: now also J9.4 (Pin_4)
- net Trip Reset: now also R1.1, SW1.2
- net at R8.1: now also U9.13 (GPIO11/TOUCH11/ADC2_CH0/FSPID/FSPIIO5)
- net at R12.1: now also U9.19 (GPIO17/U1TXD/ADC2_CH6/DAC_1)
- net at R9.1: now also U9.14 (GPIO12/TOUCH12/ADC2_CH1/FSPICLK/FSPIIO6)
- net at R10.1: now also U9.15 (GPIO13/TOUCH13/ADC2_CH2/FSPIQ/FSPIIO7)
- net at R13.1: now also U9.22 (GPIO18/U1RXD/ADC2_CH7/DAC_2/CLK_OUT3/RGB_LED)
- net at R11.1: now also U9.16 (GPIO14/TOUCH14/ADC2_CH3/FSPIWP/FSPIDQS)
- net Trigger: now reaches U9.23 (GPIO19/U1RTS/ADC2_CH8/CLK_OUT2/USB_D-)
- net Trigger: now also J7.3 (Pin_3)
- net Echo: now reaches U9.24 (GPIO20/U1CTS/ADC2_CH9/CLK_OUT1/USB_D+)
- net Echo: now also J7.2 (Pin_2)
- net LED Data Out: now reaches U9.25 (GPIO21)
- net CL: now reaches U9.29 (GPIO35)
- net CL: now also J8.3 (Pin_3)
- net DA: now reaches U9.30 (GPIO36)
- net DA: now also J8.4 (Pin_4)
- net CS: now reaches U9.31 (GPIO37)
- net CS: now also J8.5 (Pin_5)
- net DC: now reaches U9.32 (GPIO38)
- net DC: now also J8.6 (Pin_6)
- net at U9.37 (U0TXD/GPIO43/CLK_OUT1): now also LS1.1
- net at U9.38 (U0RXD/GPIO44/CLK_OUT2): now also LS1.2
- net BL: now reaches U9.39 (GPIO45/VSPI)
- net BL: now also J8.7 (Pin_7)
- net at D4.1 (DO): now also D8.4 (DI)
- net at D3.1 (DO): now also D7.4 (DI)
- net Headlights On Off renamed Headlights Low/High
- removed net Signal In: Q1.3 (D), Q2.3 (D), R25.2, R27.2
- net Signal Out renamed Speed Out
- net Speed Out: now also U9.4 (GPIO2/TOUCH2/ADC1_CH1); no longer Q2.1 (S), R26.2
- net Temp LED: no longer names the net of D2.4 (DI)
- net Temp LED: now also D11.1 (DO)
- new net: D11.4 (DI), D9.1 (DO)
- new net: D7.1 (DO), D9.4 (DI)
- new net: D10.4 (DI), D8.1 (DO)
- new net Tach Out: Q2.1 (S), R26.2, U9.3 (GPIO1/TOUCH1/ADC1_CH0)
- no-connect marks 19 -> 14
Other:
- note added: "Batt LED"
- note added: "Brake LED"
- note added: "Fuel LED"
- note added: "High Beam LED"
- note added: "Left Turn LED"
- note added: "Low Beam LED"
- note added: "Oil LED"
- note added: "Right Turn LED"
- note added: "Temp LED"
- moved on the sheet: D2, D3, D4, Q3, R10, R11, R12, R13, R40, R8, R9, U8

Commit message: Second Update
Added inputs for turn and brake lights, fixed pin positions, added connector for lights and power
Parts:
- added J10: Conn_01x03_Socket, symbol Connector:Conn_01x03_Socket
- added J9: Conn_01x05_Socket, symbol Connector:Conn_01x05_Socket
- renumbered C7 to C1, C11 to C10, C12 to C11, C13 to C12, C15 to C13, C16 to C14, C5 to C2, C6 to C5, C8 to C6, C9 to C7, C14 to C8, C10 to C9, D5 to D10, D6 to D11, D3 to D2, D7 to D3, D9 to D4, D11 to D5, D2 to D6, D4 to D7, D10 to D9, J7 to J11, J8 to J7, J9 to J8, Q3 to Q1, Q1 to Q2, Q2 to Q3, R17 to R1, R24 to R10, R25 to R11, R26 to R12, R27 to R13, R1 to R14, R8 to R15, R9 to R16, R10 to R17, R11 to R18, R12 to R19, R39 to R2, R13 to R20, R29 to R3, R32 to R4, R30 to R5, R33 to R6, R31 to R7, R34 to R8, R40 to R9, U8 to U1, U6 to U2, U7 to U3, U2 to U4, U3 to U5, U9 to U6
Connections:
- net +BATT: now also J10.2 (Pin_2)
- net +VDC: now also J10.3 (Pin_3)
- net BL: now also U6.36 (MTMS/JTAG/GPIO42); no longer U6.39 (GPIO45/VSPI)
- net CL: now also U6.39 (GPIO45/VSPI); no longer U6.29 (GPIO35)
- net CS: now also U6.34 (MTDO/JTAG/GPIO40); no longer U6.31 (GPIO37)
- net DA: now also U6.33 (MTCK/JTAG/GPIO39); no longer U6.30 (GPIO36)
- net DC: now also U6.35 (MTDI/JTAG/GPIO41); no longer U6.32 (GPIO38)
- net GND: now also J10.1 (Pin_1)
- net Ignition Sensor: now also U6.15 (GPIO13/TOUCH13/ADC2_CH2/FSPIQ/FSPIIO7); no longer U6.11 (GPIO9/TOUCH9/ADC1_CH8/FSPIHD)
- net LED Data Out: now also U6.30 (GPIO36); no longer U6.25 (GPIO21)
- net Power Off: now also U6.16 (GPIO14/TOUCH14/ADC2_CH3/FSPIWP/FSPIDQS); no longer U6.12 (GPIO10/TOUCH10/ADC1_CH9/FSPICS0/FSPIIO4)
- net SCL: now also U6.32 (GPIO38); no longer U6.28 (GPIO34)
- net SDA: now also U6.31 (GPIO37); no longer U6.27 (GPIO33)
- net at R15.1: now also U6.19 (GPIO17/U1TXD/ADC2_CH6/DAC_1); no longer U6.13 (GPIO11/TOUCH11/ADC2_CH0/FSPID/FSPIIO5)
- net at R19.1: now also U6.28 (GPIO34); no longer U6.19 (GPIO17/U1TXD/ADC2_CH6/DAC_1)
- net at R16.1: now also U6.22 (GPIO18/U1RXD/ADC2_CH7/DAC_2/CLK_OUT3/RGB_LED); no longer U6.14 (GPIO12/TOUCH12/ADC2_CH1/FSPICLK/FSPIIO6)
- net at R17.1: now also U6.25 (GPIO21); no longer U6.15 (GPIO13/TOUCH13/ADC2_CH2/FSPIQ/FSPIIO7)
- net at R20.1: now also U6.29 (GPIO35); no longer U6.22 (GPIO18/U1RXD/ADC2_CH7/DAC_2/CLK_OUT3/RGB_LED)
- net at R18.1: now also U6.27 (GPIO33); no longer U6.16 (GPIO14/TOUCH14/ADC2_CH3/FSPIWP/FSPIDQS)
- net Headlights Low/High renamed Headlights Low
- net Headlights Low: now also J9.5 (Pin_5)
- new net Brake In: J9.1 (Pin_1), U6.14 (GPIO12/TOUCH12/ADC2_CH1/FSPICLK/FSPIIO6)
- new net Headlights High: J9.4 (Pin_4), U6.11 (GPIO9/TOUCH9/ADC1_CH8/FSPIHD)
- new net Left Turn In: J9.3 (Pin_3), U6.12 (GPIO10/TOUCH10/ADC1_CH9/FSPICS0/FSPIIO4)
- new net Right Turn In: J9.2 (Pin_2), U6.13 (GPIO11/TOUCH11/ADC2_CH0/FSPID/FSPIIO5)
- no-connect marks 14 -> 10
Other:
- moved on the sheet: C1, C10, C11, C12, C13, C14, C2, C3, C4, C5, C6, C7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

Commit message: fixed misplaced file
Parts:
- removed Q2, Q3: 2N7000, Package_TO_SOT_THT:TO-92_Inline, symbol Transistor_FET:2N7000
- added Q10, Q11, Q12, Q13, Q14, Q15, Q2, Q3, Q4, Q5, Q6, Q7, Q8, Q9: NPN, symbol Simulation_SPICE:NPN
- added R21, R23, R25, R26, R27, R28, R35, R36, R37, R38, R39, R40, R43, R44: 1K, symbol Device:R
- added R22, R24, R29, R30, R31, R32, R33, R34, R41, R42: 10K, symbol Device:R
Connections:
- net +3.3V: now also R10.2, R12.2, R24.2, R29.2, R30.2, R31.2, R41.2; no longer R10.1, R12.1
- net +5V: now also R11.2, R13.2, R22.2, R32.2, R33.2, R34.2, R42.2; no longer R11.1, R13.1
- net Brake In: now also R44.1; no longer U6.14 (GPIO12/TOUCH12/ADC2_CH1/FSPICLK/FSPIIO6)
- net GND: now also Q10.3 (E), Q11.3 (E), Q12.3 (E), Q13.3 (E), Q14.3 (E), Q15.3 (E), Q2.3 (E), Q3.3 (E), Q4.3 (E), Q5.3 (E), Q6.3 (E), Q7.3 (E), Q8.3 (E), Q9.3 (E)
- net Left Turn In: now also R39.1; no longer U6.12 (GPIO10/TOUCH10/ADC1_CH9/FSPICS0/FSPIIO4)
- net Right Turn In: now also R40.1; no longer U6.13 (GPIO11/TOUCH11/ADC2_CH0/FSPID/FSPIIO5)
- net Speed In: now also R21.1; no longer R11.2
- net Speed Out: now also Q5.1 (C), R24.1; no longer R10.2
- net Tach In: now also R26.1; no longer R13.2
- net Tach Out: now also R10.1, Q2.1 (C); no longer R12.2
- net Headlights High renamed Headlights High In
- net Headlights High In: now also R38.1; no longer U6.11 (GPIO9/TOUCH9/ADC1_CH8/FSPIHD)
- net Headlights Low renamed Headlights Low In
- net Headlights Low In: now also R28.1; no longer U6.10 (GPIO8/TOUCH8/ADC1_CH7)
- new net: Q15.2 (B), R44.2
- new net: Q4.1 (C), R22.1, R23.1
- new net: Q5.2 (B), R23.2
- new net: Q8.2 (B), R35.2
- new net: Q4.2 (B), R21.2
- new net: Q6.1 (C), R11.1, R25.1
- new net: Q2.2 (B), R25.2
- new net: Q6.2 (B), R26.2
- new net: Q12.1 (C), R33.1, R36.1
- new net: Q9.2 (B), R36.2
- new net: Q13.1 (C), R34.1, R37.1
- new net: Q10.2 (B), R37.2
- new net: Q15.1 (C), R42.1, R43.1
- new net: Q7.2 (B), R28.2
- new net: Q12.2 (B), R39.2
- new net: Q11.1 (C), R32.1, R35.1
- new net: Q11.2 (B), R38.2
- new net: Q13.2 (B), R40.2
- new net: Q14.2 (B), R43.2
- new net: Q7.1 (C), R13.1, R27.1
- new net: Q3.2 (B), R27.2
- new net Brake Out: Q14.1 (C), R41.1, U6.14 (GPIO12/TOUCH12/ADC2_CH1/FSPICLK/FSPIIO6)
- new net Headlights High Out: Q8.1 (C), R29.1, U6.11 (GPIO9/TOUCH9/ADC1_CH8/FSPIHD)
- new net Headlights Low Out: Q3.1 (C), R12.1, U6.10 (GPIO8/TOUCH8/ADC1_CH7)
- new net Left Turn Out: Q9.1 (C), R30.1, U6.12 (GPIO10/TOUCH10/ADC1_CH9/FSPICS0/FSPIIO4)
- new net Right Turn Out: Q10.1 (C), R31.1, U6.13 (GPIO11/TOUCH11/ADC2_CH0/FSPID/FSPIIO5)
Other:
- moved on the sheet: LS1, R14, R15, R16, R17, R18, R19, R20, SW1, U6
