File: Dash.kicad_sch (KiCad schematic)
At the start: 89 parts, among them J1 Conn_01x03_Socket, J10 Conn_01x03_Socket, J11 Conn_01x04_Socket, J2 Conn_01x03_Socket, J3 Conn_01x03_Socket, J4 Conn_01x03_Socket, J5 Conn_01x03_Socket, J6 Conn_01x03_Socket, J7 Conn_01x07_Socket, J8 Conn_01x06_Socket, J9 Conn_01x05_Socket, Q1 2N7000, Q16 NMOS, Q17 NMOS, Q18 NMOS, Q19 NMOS, Q2 NMOS, Q20 NMOS, Q4 NMOS, Q5 NMOS, SW1 SW_Push, U1 SFH617A-1, U2 24C02Cx-x-SN, U3 24C02Cx-x-SN, U4 LM2678T-3.3, U5 LM2678T-5.0, U6 ESP32-S2-DevKitM

Commit message: Started prototype PCB layout
Parts:
- C1, C12, C5, C8: footprint (none) -> Capacitor_THT:C_Disc_D3.0mm_W1.6mm_P2.50mm
- C10, C11, C13, C14, C2, C3, C4, C6, C7, C9: footprint (none) -> Capacitor_THT:CP_Radial_D5.0mm_P2.50mm
- D10, D11, D12, D13: footprint (none) -> Diode_THT:D_A-405_P7.62mm_Horizontal
- J1, J10, J2, J3, J4, J5, J6: footprint (none) -> Connector_Molex:Molex_KK-396_A-41791-0003_1x03_P3.96mm_Vertical
- J11: footprint (none) -> Connector_Molex:Molex_KK-396_5273-04A_1x04_P3.96mm_Vertical
- J7: footprint (none) -> Connector_Molex:Molex_KK-396_5273-07A_1x07_P3.96mm_Vertical
- J8: footprint (none) -> Connector_Molex:Molex_KK-396_5273-06A_1x06_P3.96mm_Vertical
- J9: footprint (none) -> Connector_Molex:Molex_KK-396_5273-05A_1x05_P3.96mm_Vertical
- L1, L2: footprint (none) -> Inductor_THT:L_Radial_D9.5mm_P5.00mm_Fastron_07HVP
- LS1: footprint (none) -> Connector_Molex:Molex_KK-396_5273-02A_1x02_P3.96mm_Vertical
- Q16, Q17, Q18, Q19, Q2, Q20, Q4, Q5: footprint (none) -> Package_TO_SOT_THT:TO-92_Inline
- R1, R14, R15, R16, R17, R18, R19, R2, R20, R3, R4, R5, R6, R7, R8, R9: footprint (none) -> Resistor_THT:R_Axial_DIN0207_L6.3mm_D2.5mm_P10.16mm_Horizontal
- R10, R11, R21, R22, R23, R24, R45, R46, R47, R48, R49, R50, R51, R52, R53, R54: value R -> 10K; footprint (none) -> Resistor_THT:R_Axial_DIN0207_L6.3mm_D2.5mm_P10.16mm_Horizontal
- SW1: footprint (none) -> Button_Switch_THT:SW_PUSH_6mm_H8mm
- U4, U5: footprint (none) -> Package_TO_SOT_THT:TO-220-7_P2.54x3.7mm_StaggerOdd_Lead3.8mm_Vertical
- U6: footprint PCM_Espressif:ESP32-S2-DevKitM -> Espressif:ESP32-S2-DevKitM
Connections:
- no-connect marks 10 -> 11

Commit message: pin update
Updated pin assignments
Parts:
- added R12, R13: 10k, symbol Device:R
Connections:
- net +3.3V: now also R12.1, R13.1
- net BL: no longer U6.36 (MTMS/JTAG/GPIO42)
- net Brake Adjusted: now also U6.27 (GPIO33); no longer U6.14 (GPIO12/TOUCH12/ADC2_CH1/FSPICLK/FSPIIO6)
- net CL: now also U6.30 (GPIO36); no longer U6.40 (GPIO46/LOG)
- net CS: no longer U6.34 (MTDO/JTAG/GPIO40)
- net DA: now also U6.29 (GPIO35); no longer U6.33 (MTCK/JTAG/GPIO39)
- net DC: now also U6.31 (GPIO37); no longer U6.35 (MTDI/JTAG/GPIO41)
- net Echo Adjusted: now also U6.19 (GPIO17/U1TXD/ADC2_CH6/DAC_1); no longer U6.17 (GPIO15/U0RTS/ADC2_CH4/XTAL_32K_P)
- net Headlights High Adjusted: now also U6.32 (GPIO38); no longer U6.11 (GPIO9/TOUCH9/ADC1_CH8/FSPIHD)
- net Headlights Low Adjusted: now also U6.40 (GPIO46/LOG); no longer U6.10 (GPIO8/TOUCH8/ADC1_CH7)
- net Ignition Sensor: now also U6.33 (MTCK/JTAG/GPIO39); no longer U6.15 (GPIO13/TOUCH13/ADC2_CH2/FSPIQ/FSPIIO7)
- net LED Data Out: now also U6.35 (MTDI/JTAG/GPIO41); no longer U6.30 (GPIO36)
- net Left Turn Adjusted: now also U6.22 (GPIO18/U1RXD/ADC2_CH7/DAC_2/CLK_OUT3/RGB_LED); no longer U6.12 (GPIO10/TOUCH10/ADC1_CH9/FSPICS0/FSPIIO4)
- net Power Off: now also U6.34 (MTDO/JTAG/GPIO40); no longer U6.16 (GPIO14/TOUCH14/ADC2_CH3/FSPIWP/FSPIDQS)
- net Right Turn Adjusted: now also U6.25 (GPIO21); no longer U6.13 (GPIO11/TOUCH11/ADC2_CH0/FSPID/FSPIIO5)
- net SCL: now also U6.11 (GPIO9/TOUCH9/ADC1_CH8/FSPIHD); no longer U6.32 (GPIO38)
- net SDA: now also U6.10 (GPIO8/TOUCH8/ADC1_CH7); no longer U6.31 (GPIO37)
- net at R15.1: now also U6.12 (GPIO10/TOUCH10/ADC1_CH9/FSPICS0/FSPIIO4); no longer U6.19 (GPIO17/U1TXD/ADC2_CH6/DAC_1)
- net at R19.1: now also U6.16 (GPIO14/TOUCH14/ADC2_CH3/FSPIWP/FSPIDQS); no longer U6.28 (GPIO34)
- net at R16.1: now also U6.13 (GPIO11/TOUCH11/ADC2_CH0/FSPID/FSPIIO5); no longer U6.22 (GPIO18/U1RXD/ADC2_CH7/DAC_2/CLK_OUT3/RGB_LED)
- net at R17.1: now also U6.14 (GPIO12/TOUCH12/ADC2_CH1/FSPICLK/FSPIIO6); no longer U6.25 (GPIO21)
- net at R20.1: now also U6.17 (GPIO15/U0RTS/ADC2_CH4/XTAL_32K_P); no longer U6.29 (GPIO35)
- net at R18.1: now also U6.15 (GPIO13/TOUCH13/ADC2_CH2/FSPIQ/FSPIIO7); no longer U6.27 (GPIO33)
- net at LS1.1: now also U6.36 (MTMS/JTAG/GPIO42); no longer U6.38 (U0RXD/GPIO44/CLK_OUT2)
- net CS1: now reaches U6.39 (GPIO45/VSPI)
- net CS1: now also R12.2
- new net CS0: R13.2, U6.28 (GPIO34)

Commit message: Update Schematic
Reverted to older logic shifter design. Added single stage amplifier. Added voltage dividers for gauges.
Parts:
- removed Q16, Q17, Q18, Q19, Q2, Q20, Q4, Q5: NMOS, Package_TO_SOT_THT:TO-92_Inline, symbol Simulation_SPICE:NMOS
- added C15: 47uF, Capacitor_THT:CP_Radial_D5.0mm_P2.50mm, symbol Device:C_Polarized
- added Q10, Q11, Q12, Q13, Q14, Q15, Q16, Q2, Q3, Q4, Q5, Q6, Q7, Q8, Q9: NPN, symbol Simulation_SPICE:NPN
- added R25, R26, R28, R31, R35, R36, R37, R38, R39, R40, R43, R44: 1K, symbol Device:R
- added R27, R29, R30, R32, R33, R34, R41, R42: 10K, symbol Device:R
- added R55: 2K, symbol Device:R
- R10, R11, R22, R24, R45, R46: footprint Resistor_THT:R_Axial_DIN0207_L6.3mm_D2.5mm_P10.16mm_Horizontal -> (none)
- R21, R23: value 10K -> 1K; footprint Resistor_THT:R_Axial_DIN0207_L6.3mm_D2.5mm_P10.16mm_Horizontal -> (none)
- R47, R49, R50: value 10K -> 47; footprint Resistor_THT:R_Axial_DIN0207_L6.3mm_D2.5mm_P10.16mm_Horizontal -> (none)
- R48: value 10K -> 51k; footprint Resistor_THT:R_Axial_DIN0207_L6.3mm_D2.5mm_P10.16mm_Horizontal -> (none)
- R51, R53, R54: value 10K -> 10; footprint Resistor_THT:R_Axial_DIN0207_L6.3mm_D2.5mm_P10.16mm_Horizontal -> (none)
- R52: value 10K -> 10k; footprint Resistor_THT:R_Axial_DIN0207_L6.3mm_D2.5mm_P10.16mm_Horizontal -> (none)
Connections:
- net +3.3V: now also R10.2, R24.2, R45.2, R46.2, R29.2, R30.2, R41.2; no longer R10.1, R21.1, R23.1, R45.1, R47.1, R49.1, R51.1, R53.1
- net +5V: now also R11.2, R22.2, R47.1, R49.1, R27.2, R32.2, R33.2, R34.2, R42.2; no longer R11.1, R22.1, R24.1, R46.1, R48.1, R52.1, R54.1
- net Batt In: no longer U6.6 (GPIO4/TOUCH4/ADC1_CH3)
- net Brake Adjusted: no longer R51.2
- net Brake In: now also R44.1; no longer R52.2
- net Echo Adjusted: no longer R10.2
- net Echo In: no longer R11.2
- net Fuel In: now also R53.2; no longer U6.7 (GPIO5/TOUCH5/ADC1_CH4)
- net GND: now also R52.2, Q10.3 (E), Q11.3 (E), Q12.3 (E), Q13.3 (E), Q14.3 (E), Q15.3 (E), Q16.3 (E), Q2.3 (E), Q3.3 (E), Q4.3 (E), Q5.3 (E), Q6.3 (E), Q7.3 (E), Q8.3 (E), Q9.3 (E); no longer LS1.2
- net Headlights High Adjusted: no longer R23.2
- net Headlights High In: now also R38.1; no longer R24.2
- net Headlights Low Adjusted: no longer R53.2
- net Headlights Low In: now also R28.1; no longer R54.2
- net Left Turn Adjusted: no longer R47.2
- net Left Turn In: now also R39.1; no longer R48.2
- net Oil In: now also R54.2; no longer U6.8 (GPIO6/TOUCH6/ADC1_CH5)
- net Right Turn Adjusted: no longer R49.2
- net Right Turn In: now also R40.1; no longer R50.2
- net Speed Adjusted: no longer R45.2
- net Speed In: now also R21.1; no longer R46.2
- net Tach Adjusted: no longer R21.2
- net Tach In: now also R26.1; no longer R22.2
- net Temp In: now also R51.2; no longer U6.5 (GPIO3/TOUCH3/ADC1_CH2)
- net VAA: now also LS1.1, R48.1
- net Speaker Signal: now reaches U6.36 (MTMS/JTAG/GPIO42)
- net Speaker Signal: now also C15.1; no longer LS1.1
- new net: R50.2, R54.1, U6.8 (GPIO6/TOUCH6/ADC1_CH5)
- new net: Q9.2 (B), R36.2
- new net: R48.2, R52.1, U6.6 (GPIO4/TOUCH4/ADC1_CH3)
- new net: Q8.2 (B), R35.2
- new net: Q7.2 (B), R28.2
- new net: C15.2, Q16.2 (B), R55.1
- new net: LS1.2, Q16.1 (C), R55.2
- new net: Q11.1 (C), R32.1, R35.1
- new net: Q10.2 (B), R37.2
- new net: Q13.1 (C), R34.1, R37.1
- new net: Q7.1 (C), R27.1, R31.1
- new net: Q4.1 (C), R22.1, R23.1
- new net: Q13.2 (B), R40.2
- new net: Q12.1 (C), R33.1, R36.1
- new net: Q14.2 (B), R43.2
- new net: Q4.2 (B), R21.2
- new net: Q2.2 (B), R25.2
- new net: R47.2, R51.1, U6.5 (GPIO3/TOUCH3/ADC1_CH2)
- new net: Q15.1 (C), R42.1, R43.1
- new net: Q15.2 (B), R44.2
- new net: Q11.2 (B), R38.2
- new net: Q6.1 (C), R11.1, R25.1
- new net: Q6.2 (B), R26.2
- new net: Q3.2 (B), R31.2
- new net: Q12.2 (B), R39.2
- new net: R49.2, R53.1, U6.7 (GPIO5/TOUCH5/ADC1_CH4)
- new net: Q5.2 (B), R23.2
- new net Brake Out: Q14.1 (C), R41.1
- new net Headlights High Out: Q8.1 (C), R29.1
- new net Headlights Low Out: Q3.1 (C), R45.1
- new net Left Turn Out: Q9.1 (C), R30.1
- new net Right Turn Out: Q10.1 (C), R46.1
- new net Speed Out: Q5.1 (C), R24.1
- new net Tach Out: Q2.1 (C), R10.1
Other:
- moved on the sheet: LS1, R12, R13, R15, R16, R17, R18, R19, R20, U6
