File: Dash.kicad_sch (KiCad schematic)
At the start: 120 parts, among them J1 Conn_01x03_Socket, J10 Conn_01x03_Socket, J11 Conn_01x04_Socket, J2 Conn_01x03_Socket, J3 Conn_01x03_Socket, J4 Conn_01x03_Socket, J5 Conn_01x03_Socket, J6 Conn_01x03_Socket, J7 Conn_01x07_Socket, J8 Conn_01x06_Socket, J9 Conn_01x05_Socket, Q1 2N7000, Q10 NPN, Q11 NPN, Q12 NPN, Q13 NPN, Q14 NPN, Q15 NPN, Q16 NPN, Q17 NPN, Q18 NPN, Q2 NPN, Q3 NPN, Q4 NPN, Q5 NPN, Q6 NPN, Q7 NPN, Q8 NPN, Q9 NPN, SW1 SW_Push, U1 SFH617A-1, U2 24C02Cx-x-SN, U3 24C02Cx-x-SN, U4 ADS1015IDGS, U5 LM2678T-5.0, U6 ESP32-S2-DevKitM

Commit message: Update Dash.kicad_sch
Removed servo motors. Added drivers and shift registers for stepper motors
Parts:
- removed J1, J2, J3, J4, J5, J6: Conn_01x03_Socket, Connector_Molex:Molex_KK-396_A-41791-0003_1x03_P3.96mm_Vertical, symbol Connector:Conn_01x03_Socket
- removed R16, R17, R18, R19: 220, Resistor_THT:R_Axial_DIN0207_L6.3mm_D2.5mm_P10.16mm_Horizontal, symbol Device:R
- added C21, C22, C23, C24, C25, C26, C27, C28, C29, C30, C31, C32, C33, C34, C35: 100n, Capacitor_THT:C_Disc_D3.0mm_W1.6mm_P2.50mm, symbol Device:C
- added J13, J14, J15, J16, J17, J18: Conn_01x04_Socket, Connector_Hirose:Hirose_DF13-04P-1.25DSA_1x04_P1.25mm_Vertical, symbol Connector:Conn_01x04_Socket
- added R63, R64, R65: 10K, Resistor_THT:R_Axial_DIN0207_L6.3mm_D2.5mm_P10.16mm_Horizontal, symbol Device:R
- added U10, U11, U9: 74HC595, Package_DIP:DIP-16_W7.62mm, symbol 74xx:74HC595
- added U12, U13, U14, U15, U16, U17: L293D, Package_DIP:DIP-16_W7.62mm, symbol Driver_Motor:L293D
- R15: value 220 -> 10k; footprint Resistor_THT:R_Axial_DIN0207_L6.3mm_D2.5mm_P10.16mm_Horizontal -> (none)
Connections:
- net +3.3V: now also R15.1
- net +5V: now also C21.1, C22.1, C23.1, C24.1, C25.1, C26.1, C27.1, C28.1, C29.1, C30.1, C31.1, C32.1, C33.1, C34.1, C35.1, R63.1, R64.1, R65.1, U10.10 (~{SRCLR}), U10.16 (VCC), U11.10 (~{SRCLR}), U11.16 (VCC), U12.1 (EN1,2), U12.16 (VCC1), U12.8 (VCC2), U12.9 (EN3,4), U13.1 (EN1,2), U13.16 (VCC1), U13.8 (VCC2), U13.9 (EN3,4), U14.1 (EN1,2), U14.16 (VCC1), U14.8 (VCC2), U14.9 (EN3,4), U15.1 (EN1,2), U15.16 (VCC1), U15.8 (VCC2), U15.9 (EN3,4), U16.1 (EN1,2), U16.16 (VCC1), U16.8 (VCC2), U16.9 (EN3,4), U17.1 (EN1,2), U17.16 (VCC1), U17.8 (VCC2), U17.9 (EN3,4), U9.10 (~{SRCLR}), U9.16 (VCC)
- net CL: now also U10.11 (SRCLK), U11.11 (SRCLK), U9.11 (SRCLK)
- net DA: now also U9.14 (SER)
- net GND: now also C21.2, C22.2, C23.2, C24.2, C25.2, C26.2, C27.2, C28.2, C29.2, C30.2, C31.2, C32.2, C33.2, C34.2, C35.2, U10.8 (GND), U11.8 (GND), U12.12 (GND), U12.13 (GND), U12.4 (GND), U12.5 (GND), U13.12 (GND), U13.13 (GND), U13.4 (GND), U13.5 (GND), U14.12 (GND), U14.13 (GND), U14.4 (GND), U14.5 (GND), U15.12 (GND), U15.13 (GND), U15.4 (GND), U15.5 (GND), U16.12 (GND), U16.13 (GND), U16.4 (GND), U16.5 (GND), U17.12 (GND), U17.13 (GND), U17.4 (GND), U17.5 (GND), U9.8 (GND)
- net at U6.12 (GPIO10/TOUCH10/ADC1_CH9/FSPICS0/FSPIIO4): no longer R15.1
- net Oil_Servo renamed CS2
- net CS2: now also U10.12 (RCLK), U11.12 (RCLK), U9.12 (RCLK)
- new net: R63.2, U9.13 (~{OE})
- new net: R64.2, U10.13 (~{OE})
- new net: J17.1 (Pin_1), U12.3 (1Y)
- new net: J17.2 (Pin_2), U12.6 (2Y)
- new net: J17.3 (Pin_3), U12.11 (3Y)
- new net: J17.4 (Pin_4), U12.14 (4Y)
- new net: J15.1 (Pin_1), U14.3 (1Y)
- new net: J15.2 (Pin_2), U14.6 (2Y)
- new net: J15.3 (Pin_3), U14.11 (3Y)
- new net: J15.4 (Pin_4), U14.14 (4Y)
- new net: U10.6 (QG), U15.10 (3A)
- new net: J16.3 (Pin_3), U15.11 (3Y)
- new net: J16.4 (Pin_4), U15.14 (4Y)
- new net: U10.7 (QH), U15.15 (4A)
- new net: U10.4 (QE), U15.2 (1A)
- new net: J16.1 (Pin_1), U15.3 (1Y)
- new net: J16.2 (Pin_2), U15.6 (2Y)
- new net: U10.5 (QF), U15.7 (2A)
- new net: U11.6 (QG), U17.10 (3A)
- new net: J14.3 (Pin_3), U17.11 (3Y)
- new net: J14.4 (Pin_4), U17.14 (4Y)
- new net: U11.7 (QH), U17.15 (4A)
- new net: U11.4 (QE), U17.2 (1A)
- new net: J14.1 (Pin_1), U17.3 (1Y)
- new net: J14.2 (Pin_2), U17.6 (2Y)
- new net: U11.5 (QF), U17.7 (2A)
- new net: J13.1 (Pin_1), U16.3 (1Y)
- new net: J13.2 (Pin_2), U16.6 (2Y)
- new net: J13.3 (Pin_3), U16.11 (3Y)
- new net: J13.4 (Pin_4), U16.14 (4Y)
- new net: U10.2 (QC), U14.10 (3A)
- new net: U10.3 (QD), U14.15 (4A)
- new net: U10.15 (QA), U14.2 (1A)
- new net: U10.1 (QB), U14.7 (2A)
- new net: U11.1 (QB), U16.7 (2A)
- new net: R65.2, U11.13 (~{OE})
- new net: U10.9 (QH'), U11.14 (SER)
- new net: U11.15 (QA), U16.2 (1A)
- new net: U11.2 (QC), U16.10 (3A)
- new net: U11.3 (QD), U16.15 (4A)
- new net: U12.7 (2A), U9.1 (QB)
- new net: U12.2 (1A), U9.15 (QA)
- new net: U12.10 (3A), U9.2 (QC)
- new net: U12.15 (4A), U9.3 (QD)
- new net: U13.2 (1A), U9.4 (QE)
- new net: U13.7 (2A), U9.5 (QF)
- new net: U13.10 (3A), U9.6 (QG)
- new net: U13.15 (4A), U9.7 (QH)
- new net: U10.14 (SER), U9.9 (QH')
- new net: J18.3 (Pin_3), U13.11 (3Y)
- new net: J18.4 (Pin_4), U13.14 (4Y)
- new net: J18.1 (Pin_1), U13.3 (1Y)
- new net: J18.2 (Pin_2), U13.6 (2Y)
- no-connect marks 13 -> 14

Commit message: update
Parts:
- removed R20: 220, Resistor_THT:R_Axial_DIN0207_L6.3mm_D2.5mm_P10.16mm_Horizontal, symbol Device:R
- renumbered C9 to C1, C23 to C10, C15 to C11, C25 to C12, C24 to C13, C32 to C14, C33 to C15, C27 to C16, C26 to C17, C31 to C18, C34 to C19, C10 to C2, C29 to C20, C28 to C21, C30 to C22, C35 to C23, C11 to C3, C12 to C4, C8 to C5, C13 to C6, C14 to C7, C21 to C8, C22 to C9, D11 to D1, D7 to D10, D8 to D11, D9 to D12, D1 to D2, D12 to D3, D13 to D4, D2 to D5, D3 to D6, D4 to D7, D5 to D8, D6 to D9, J7 to J1, J13 to J10, J14 to J11, J8 to J2, J9 to J3, J10 to J4, J11 to J5, J17 to J6, J18 to J7, J15 to J8, J16 to J9, L2 to L1, Q4 to Q1, Q2 to Q10, Q9 to Q11, Q18 to Q12, Q7 to Q13, Q13 to Q14, Q3 to Q15, Q10 to Q16, Q1 to Q17, Q16 to Q18, Q11 to Q2, Q15 to Q3, Q5 to Q4, Q8 to Q5, Q14 to Q6, Q6 to Q7, Q12 to Q8, Q17 to Q9, R21 to R1, R24 to R10, R29 to R11, R41 to R12, R26 to R13, R39 to R14, R56 to R15, R11 to R16, R33 to R17, R57 to R18, R25 to R19, R38 to R2, R36 to R20, R58 to R21, R10 to R22, R30 to R23, R59 to R24, R28 to R25, R40 to R26, R34 to R28, R47 to R29, R44 to R3, R51 to R30, R37 to R32, R48 to R33, R52 to R34, R45 to R35, R46 to R36, R49 to R37, R53 to R38, R50 to R39, R22 to R4, R54 to R40, R9 to R41, R15 to R42, R3 to R43, R5 to R44, R7 to R45, R1 to R46, R4 to R47, R6 to R48, R8 to R49, R32 to R5, R63 to R50, R64 to R51, R65 to R52, R2 to R53, R12 to R54, R13 to R55, R55 to R56, R14 to R57, R42 to R6, R23 to R7, R35 to R8, R43 to R9, U5 to U1, U12 to U10, U13 to U11, U14 to U12, U15 to U13, U16 to U14, U17 to U15, U4 to U2, U1 to U3, U2 to U4, U6 to U5, U3 to U6, U9 to U7, U10 to U8, U11 to U9
Connections:
- net CS2: now also U5.17 (GPIO15/U0RTS/ADC2_CH4/XTAL_32K_P)
- no-connect marks 14 -> 19
Other:
- moved on the sheet: C10, C12, C13, C14, C15, C16, C17, C18, C19, C20, C21, C22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

Commit message: update on off
Parts:
- removed D3, D4: D, Diode_THT:D_A-405_P7.62mm_Horizontal, symbol Device:D
- removed J1: Conn_01x07_Socket, Connector_Molex:Molex_KK-396_5273-07A_1x07_P3.96mm_Vertical, symbol Connector:Conn_01x07_Socket
- removed J3: Conn_01x05_Socket, Connector_Molex:Molex_KK-396_5273-05A_1x05_P3.96mm_Vertical, symbol Connector:Conn_01x05_Socket
- removed Q17: 2N7000, Package_TO_SOT_THT:TO-92_Inline, symbol Transistor_FET:2N7000
- removed U3: SFH617A-1, Package_DIP:DIP-4_W7.62mm, symbol Isolator:SFH617A-1
- added C24: 100n, symbol Device:C
- added D13, D14: D_Zener, symbol Device:D_Zener
- added D15, D16: D, Diode_THT:D_A-405_P7.62mm_Horizontal, symbol Device:D
- added J12, J13, J14, J15: Conn_01x06_Socket, symbol Connector:Conn_01x06_Socket
- added Q17, Q21: NPN, symbol Simulation_SPICE:NPN
- added Q19: PMOS, symbol Simulation_SPICE:PMOS
- added Q20: NMOS, symbol Simulation_SPICE:NMOS
- added R58, R60: 100k, symbol Device:R
- added R59, R61, R63: 10k, symbol Device:R
- added R62: 1k, Resistor_THT:R_Axial_DIN0207_L6.3mm_D2.5mm_P10.16mm_Horizontal, symbol Device:R
- added R64, R66: 10K, symbol Device:R
- added R65: 1K, symbol Device:R
- added U16: SFH617A-1, Package_DIP:DIP-4_W7.62mm, symbol Isolator:SFH617A-1
- R41: value 150 -> 1K; footprint Resistor_THT:R_Axial_DIN0207_L6.3mm_D2.5mm_P10.16mm_Horizontal -> (none)
Connections:
- net +3.3V: now also R66.2, U16.4
- net +5V: now also J13.2 (Pin_2), J14.2 (Pin_2), J15.2 (Pin_2), R64.2
- net +BATT: now also C24.1, D13.1 (K), Q19.3 (S), R58.1
- net +VDC: now also U16.1
- net Brake In: now also J12.1 (Pin_1)
- net CL: now also J13.3 (Pin_3), J14.3 (Pin_3), J15.3 (Pin_3)
- net CS0: now also J15.5 (Pin_5)
- net CS1: now also J14.5 (Pin_5)
- net CS2: now also J13.5 (Pin_5)
- net DA: now also J13.4 (Pin_4), J14.4 (Pin_4), J15.4 (Pin_4)
- net DC: now also J13.6 (Pin_6), J14.6 (Pin_6), J15.6 (Pin_6)
- net Echo Adjusted: now also Q21.1 (C), R66.1
- net Echo In: now also R41.1
- net GND: now also D14.2 (A), J13.1 (Pin_1), J14.1 (Pin_1), J15.1 (Pin_1), Q17.3 (E), Q20.3 (S), Q21.3 (E), R60.2, R62.2, R63.1; no longer R41.2
- net Hazard In: now also J12.6 (Pin_6)
- net Headlights High In: now also J12.4 (Pin_4)
- net Headlights Low In: now also J12.5 (Pin_5)
- net Ignition Sensor: now also R63.2, U16.3
- net Left Turn In: now also J12.3 (Pin_3)
- net Power Off: now also D16.2 (A)
- net Right Turn In: now also J12.2 (Pin_2)
- net VAA: now also Q19.1 (D)
- new net: D14.1 (K), Q20.2 (G), R60.1, R61.1
- new net: C24.2, D13.2 (A), Q19.2 (G), R58.2, R59.1
- new net: D15.1 (K), D16.1 (K), R61.2
- new net: Q20.1 (D), R59.2
- new net: Q21.2 (B), R65.2
- new net: D15.2 (A), R62.1, U16.2
- new net: Q17.1 (C), R64.1, R65.1
- new net: Q17.2 (B), R41.2
Other:
- note added: "Constant Power In"
- note added: "Out to 12v-5v Regulator"
- note added: "Switched Power In"
- moved on the sheet: C11, LS1, Q18, R29, R30, R33, R34, R37, R38, R39, R40, R43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

Commit message: update power latch
Parts:
- removed C24: 100n, symbol Device:C
- removed D13, D14: D_Zener, symbol Device:D_Zener
- removed R58: 100k, symbol Device:R
- R60: value 100k -> 47k
- R61: value 10k -> 1k
Connections:
- net +BATT: now also R59.1
- net at Q19.2 (G): now also Q20.1 (D), R59.2; no longer R59.1
Other:
- moved on the sheet: Q19, Q20, R59, R60

Commit message: Update Dash.kicad_sch
Parts:
- removed R50, R51, R52: 10K, Resistor_THT:R_Axial_DIN0207_L6.3mm_D2.5mm_P10.16mm_Horizontal, symbol Device:R
Connections:
- net GND: now also U7.13 (~{OE}), U8.13 (~{OE}), U9.13 (~{OE})

Commit message: Update Dash.kicad_sch
Connections:
- net +BATT: now also R59.2; no longer R59.1
- net at Q19.2 (G), Q20.1 (D): now also R59.1; no longer R59.2
Other:
- moved on the sheet: D15, D16, Q20, R59, R60, R61, R62, R63, U16
