File: amplifier.kicad_sch (KiCad schematic)
At the start: 4 parts, among them U8 LM7171xIM

Commit message: update
Parts:
- U8: footprint Package_SO:SOIC-8_3.9x4.9mm_P1.27mm -> Package_DIP:DIP-8_W7.62mm
Changed lines of the file:
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@@
 			)
 		)
-		(property "Footprint" "Package_SO:SOIC-8_3.9x4.9mm_P1.27mm"
+		(property "Footprint" "Package_DIP:DIP-8_W7.62mm"
 			(at 90.17 62.23 0)
 			(hide yes)
