File: eeprom.kicad_sch (KiCad schematic)
At the start: 8 parts, among them U6 24C02Cx-x-SN, U7 24C02Cx-x-SN

Commit message: update
Parts:
- U6, U7: footprint Package_SO:SOIC-8_3.9x4.9mm_P1.27mm -> Package_DIP:DIP-8_W7.62mm
Changed lines of the file:
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@@
 			)
 		)
-		(property "Footprint" "Package_SO:SOIC-8_3.9x4.9mm_P1.27mm"
+		(property "Footprint" "Package_DIP:DIP-8_W7.62mm"
 			(at 115.57 96.52 0)
 			(hide yes)
@@
 			)
 		)
-		(property "Footprint" "Package_SO:SOIC-8_3.9x4.9mm_P1.27mm"
+		(property "Footprint" "Package_DIP:DIP-8_W7.62mm"
 			(at 173.99 96.52 0)
 			(hide yes)
