File: usb.kicad_sch (KiCad schematic)
At the start: 17 parts, among them J12 USB_C_Receptacle_USB2.0_14P, Q20 NPN, Q21 NPN, U4 CP2102N-Axx-xQFN28

Commit message: update
Connections:
- net USBDN renamed USB_D_N
- net USBDP renamed USB_D_P
Changed lines of the file:
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@@
 		)
 	)
-	(label "USBDP"
+	(label "USB_D_P"
 		(at 64.77 60.96 0)
 		(effects
@@
 		)
 	)
-	(label "USBDP"
+	(label "USB_D_P"
 		(at 167.64 53.34 0)
 		(effects
@@
 		)
 	)
-	(label "USBDN"
+	(label "USB_D_N"
 		(at 167.64 50.8 0)
 		(effects
@@
 		)
 	)
-	(label "USBDN"
+	(label "USB_D_N"
 		(at 80.01 55.88 0)
 		(effects
