File: Instrument Panel Final.kicad_pcb (KiCad board)
At the start: 2 copper layers, 401.2 x 87.2 mm, 110 parts, among them IC1 LM2678SD-5.0_NOPB, J1 Conn_01x03_Socket, J10 Conn_01x07_Socket, J11 Conn_01x03_Socket, J12 Conn_01x04_Socket, J13 Conn_01x02_Socket, J14 Conn_01x03_Socket, J15 Conn_01x03_Socket, J16 USB_C_Receptacle_USB2.0_14P, J2 Conn_01x07_Socket, J3 Conn_01x07_Socket, J4 Conn_01x03_Socket, J5 Conn_01x06_Socket, J6 Conn_01x03_Socket, J7 Conn_01x05_Socket, J8 Conn_01x03_Socket, J9 Conn_01x03_Socket, Q1 NMOS, Q10 NPN, Q11 NPN, Q2 NMOS, Q3 NMOS, Q4 NMOS, Q5 NMOS, Q6 NMOS, Q7 NMOS, Q8 NMOS, Q9 2N7000, SW1 SW_Push, U1 UA78M33QDCYRQ1, U2 SFH617A-1, U3 ESP32-S3-MINI-1U, U4 24C02Cx-x-SN, U5 24C02Cx-x-SN, U6 CP2102N-Axx-xQFN28, U7 LM7171xIM

Commit message: updated to latest version
Parts:
- removed F1: AHEF750, Fuse:Fuse_Littelfuse-LVR100
- removed J13: Conn_01x02_Socket, Connector_Molex:Molex_KK-254_AE-6410-02A_1x02_P2.54mm_Vertical
- removed J14, J15: Conn_01x03_Socket, Connector_Molex:Molex_KK-396_A-41791-0003_1x03_P3.96mm_Vertical
- removed J16: USB_C_Receptacle_USB2.0_14P, Connector_USB:USB_C_Receptacle_GCT_USB4085
- added C18: 10uF, Capacitor_THT:C_Disc_D3.0mm_W1.6mm_P2.50mm, F.Cu at (171.5, 271.1)
- added C19: 0.1u, Capacitor_THT:C_Disc_D3.0mm_W1.6mm_P2.50mm, F.Cu at (393.0, 204.7)
- added C20: 1000u, Capacitor_THT:CP_Radial_D5.0mm_P2.50mm, F.Cu at (393.6, 199.8)
- added D16: APA-106-F5, LED_THT:LED_D5.0mm-4_RGB, F.Cu at (269.2, 197.5)
- added FB1: FerriteBead_Small, Inductor_THT:L_Axial_L5.0mm_D3.6mm_P10.00mm_Horizontal_Murata_BL01RN1A2A2, F.Cu at (171.5, 261.9)
- added FB2: FerriteBead_Small, Inductor_THT:L_Axial_L5.0mm_D3.6mm_P10.00mm_Horizontal_Murata_BL01RN1A2A2, F.Cu at (171.5, 267.0)
- added Q12: NPN, Package_TO_SOT_THT:TO-92_Inline, F.Cu at (257.2, 158.5)
- added Q13: NPN, Package_TO_SOT_THT:TO-92_Inline, F.Cu at (281.3, 158.5)
- added Q14: NPN, Package_TO_SOT_THT:TO-92_Inline, F.Cu at (299.0, 158.5)
- added Q15: NPN, Package_TO_SOT_THT:TO-92_Inline, F.Cu at (250.7, 158.5)
- added Q16: NPN, Package_TO_SOT_THT:TO-92_Inline, F.Cu at (274.8, 158.4)
- added Q17: NPN, Package_TO_SOT_THT:TO-92_Inline, F.Cu at (293.5, 158.5)
- added Q18: NPN, Package_TO_SOT_THT:TO-92_Inline, F.Cu at (245.2, 158.5)
- added Q19: NPN, Package_TO_SOT_THT:TO-92_Inline, F.Cu at (269.3, 158.4)
- added Q20: NPN, Package_TO_SOT_THT:TO-92_Inline, F.Cu at (516.0, 272.8)
- added Q21: NPN, Package_TO_SOT_THT:TO-92_Inline, F.Cu at (516.0, 278.6)
- added R41: 10K, Resistor_THT:R_Axial_DIN0207_L6.3mm_D2.5mm_P10.16mm_Horizontal, F.Cu at (251.2, 155.4)
- added R42: 10K, Resistor_THT:R_Axial_DIN0207_L6.3mm_D2.5mm_P10.16mm_Horizontal, F.Cu at (275.3, 155.3)
- added R43: 1K, Resistor_THT:R_Axial_DIN0207_L6.3mm_D2.5mm_P10.16mm_Horizontal, F.Cu at (290.4, 145.1)
- added R44: 1K, Resistor_THT:R_Axial_DIN0207_L6.3mm_D2.5mm_P10.16mm_Horizontal, F.Cu at (241.9, 145.3)
- added R45: 1K, Resistor_THT:R_Axial_DIN0207_L6.3mm_D2.5mm_P10.16mm_Horizontal, F.Cu at (266.3, 145.1)
- added R46: 10K, Resistor_THT:R_Axial_DIN0207_L6.3mm_D2.5mm_P10.16mm_Horizontal, F.Cu at (293.4, 155.3)
- added R47: 10K, Resistor_THT:R_Axial_DIN0207_L6.3mm_D2.5mm_P10.16mm_Horizontal, F.Cu at (245.0, 155.4)
- added R48: 10K, Resistor_THT:R_Axial_DIN0207_L6.3mm_D2.5mm_P10.16mm_Horizontal, F.Cu at (269.3, 155.3)
- added R49: 10K, Resistor_THT:R_Axial_DIN0207_L6.3mm_D2.5mm_P10.16mm_Horizontal, F.Cu at (502.2, 271.6)
- added R50: 10K, Resistor_THT:R_Axial_DIN0207_L6.3mm_D2.5mm_P10.16mm_Horizontal, F.Cu at (502.2, 275.6)
- added R51: 22.1K, Resistor_THT:R_Axial_DIN0207_L6.3mm_D2.5mm_P10.16mm_Horizontal, F.Cu at (502.2, 279.6)
- added R52: 47.5K, Resistor_THT:R_Axial_DIN0207_L6.3mm_D2.5mm_P10.16mm_Horizontal, F.Cu at (502.2, 283.7)
- added R53: 1K, Resistor_THT:R_Axial_DIN0207_L6.3mm_D2.5mm_P10.16mm_Horizontal, F.Cu at (502.2, 287.8)
- added R54: 11K, Resistor_THT:R_Axial_DIN0207_L6.3mm_D2.5mm_P10.16mm_Horizontal, F.Cu at (502.2, 291.8)
- added R55: 10K, Resistor_THT:R_Axial_DIN0207_L6.3mm_D2.5mm_P10.16mm_Horizontal, F.Cu at (502.0, 77.2)
- added R56: 10K, Resistor_THT:R_Axial_DIN0207_L6.3mm_D2.5mm_P10.16mm_Horizontal, F.Cu at (502.0, 81.3)
- added R57: 10K, Resistor_THT:R_Axial_DIN0207_L6.3mm_D2.5mm_P10.16mm_Horizontal, F.Cu at (502.0, 85.3)
- added R58: 10K, Resistor_THT:R_Axial_DIN0207_L6.3mm_D2.5mm_P10.16mm_Horizontal, F.Cu at (502.0, 89.4)
- added R59: 10K, Resistor_THT:R_Axial_DIN0207_L6.3mm_D2.5mm_P10.16mm_Horizontal, F.Cu at (502.0, 93.5)
- added R60: 10K, Resistor_THT:R_Axial_DIN0207_L6.3mm_D2.5mm_P10.16mm_Horizontal, F.Cu at (502.0, 97.5)
- added R61: 10, Resistor_THT:R_Axial_DIN0207_L6.3mm_D2.5mm_P10.16mm_Horizontal, F.Cu at (384.6, 194.5)
- added R62: 10K, Resistor_THT:R_Axial_DIN0207_L6.3mm_D2.5mm_P10.16mm_Horizontal, F.Cu at (334.1, 243.4)
- added SW2: SW_Push, Button_Switch_THT:SW_PUSH_6mm_H8mm, F.Cu at (334.5, 247.4)
- added SW3: SW_Push, Button_Switch_THT:SW_PUSH_6mm_H8mm, F.Cu at (334.5, 256.0)
- added U8: LM7171xIM, Package_SO:SOIC-8_3.9x4.9mm_P1.27mm, F.Cu at (387.2, 199.9)
- C15: value 0.1u -> 10u
- C16: value 10u -> 10uF
- C17: value 1000u -> 0.1uF; footprint Capacitor_THT:CP_Radial_D5.0mm_P2.50mm -> Capacitor_THT:C_Disc_D3.0mm_W1.6mm_P2.50mm
- C2: value 15uF -> 0.33u
- C4: value 0.47uF -> 15uF; footprint Capacitor_THT:C_Disc_D3.0mm_W1.6mm_P2.50mm -> Capacitor_THT:CP_Radial_D5.0mm_P2.50mm
- C5: value 0.33u -> 0.1u; footprint Capacitor_THT:CP_Radial_D5.0mm_P2.50mm -> Capacitor_THT:C_Disc_D3.0mm_W1.6mm_P2.50mm
- C6: value 0.1u -> 0.47uF
- D10, D8: value SMAJ5.0CA -> APA-106-F5; footprint Diode_SMD:D_SMA -> LED_THT:LED_D5.0mm-4_RGB
- D11: value 1N5819 -> APA-106-F5; footprint Diode_THT:D_DO-41_SOD81_P10.16mm_Horizontal -> LED_THT:LED_D5.0mm-4_RGB
- D14: value D_Schottky -> APA-106-F5; footprint Diode_THT:D_A-405_P7.62mm_Horizontal -> LED_THT:LED_D5.0mm-4_RGB
- D15: value SMAJ20A -> APA-106-F5; footprint Diode_SMD:D_SMA -> LED_THT:LED_D5.0mm-4_RGB
- D2: value APA-106-F5 -> D; footprint LED_THT:LED_D5.0mm-4_RGB -> Diode_THT:D_A-405_P7.62mm_Horizontal
- D4: value D -> SMAJ5.0CA; footprint Diode_THT:D_A-405_P7.62mm_Horizontal -> Diode_SMD:D_SMA
- D5, D6: value APA-106-F5 -> SMAJ5.0CA; footprint LED_THT:LED_D5.0mm-4_RGB -> Diode_SMD:D_SMA
- D7: value SMAJ5.0CA -> 1N5819; footprint Diode_SMD:D_SMA -> Diode_THT:D_DO-41_SOD81_P10.16mm_Horizontal
- J1, J4, J8: footprint Connector_Molex:Molex_KK-396_A-41791-0003_1x03_P3.96mm_Vertical -> Connector_Hirose:Hirose_DF13-03P-1.25DSA_1x03_P1.25mm_Vertical
- J10: value Conn_01x07_Socket -> Conn_01x06_Socket; footprint Connector_Molex:Molex_KK-396_5273-07A_1x07_P3.96mm_Vertical -> Connector_Hirose:Hirose_DF13-06P-1.25DSA_1x06_P1.25mm_Vertical
- J11: value Conn_01x03_Socket -> Conn_01x06_Socket; footprint Connector_Molex:Molex_KK-396_A-41791-0003_1x03_P3.96mm_Vertical -> Connector_Hirose:Hirose_DF13-06P-1.25DSA_1x06_P1.25mm_Vertical
- J12: value Conn_01x04_Socket -> USB_C_Receptacle_USB2.0_14P; footprint Connector_Molex:Molex_KK-396_5273-04A_1x04_P3.96mm_Vertical -> Connector_USB:USB_C_Receptacle_GCT_USB4085; moved to F.Cu
- J2: value Conn_01x07_Socket -> Conn_01x02_Socket; footprint Connector_Molex:Molex_KK-396_5273-07A_1x07_P3.96mm_Vertical -> Connector_Hirose:Hirose_DF13-02P-1.25DSA_1x02_P1.25mm_Vertical
- J3: value Conn_01x07_Socket -> Conn_01x03_Socket; footprint Connector_Molex:Molex_KK-396_5273-07A_1x07_P3.96mm_Vertical -> Connector_Hirose:Hirose_DF13-03P-1.25DSA_1x03_P1.25mm_Vertical
- J5: value Conn_01x06_Socket -> Conn_01x03_Socket; footprint Connector_Molex:Molex_KK-396_5273-06A_1x06_P3.96mm_Vertical -> Connector_Hirose:Hirose_DF13-03P-1.25DSA_1x03_P1.25mm_Vertical; moved to F.Cu
- J6: value Conn_01x03_Socket -> Conn_01x23_Socket; footprint Connector_Molex:Molex_KK-396_A-41791-0003_1x03_P3.96mm_Vertical -> Connector_Molex:Molex_SL_171971-0023_1x23_P2.54mm_Vertical; moved to B.Cu
- J7: value Conn_01x05_Socket -> Conn_01x03_Socket; footprint Connector_Molex:Molex_KK-396_5273-05A_1x05_P3.96mm_Vertical -> Connector_Hirose:Hirose_DF13-03P-1.25DSA_1x03_P1.25mm_Vertical; moved to F.Cu
- J9: footprint Connector_Molex:Molex_KK-396_A-41791-0003_1x03_P3.96mm_Vertical -> Connector_Hirose:Hirose_DF13-03P-1.25DSA_1x03_P1.25mm_Vertical; moved to F.Cu
- Q1: value NMOS -> 2N7000
- Q2, Q3, Q4, Q5, Q6, Q7, Q8: value NMOS -> NPN
- Q9: value 2N7000 -> NPN
- R1: value 10K -> 150
- R10, R11, R6, R7, R8, R9: value 10K -> 220
- R12, R3, R4, R5: value 10K -> 10k
- R13, R14, R15, R19, R25, R31, R32, R33, R38: value 10K -> 1K
- R18: value 150 -> 10K
- R20, R21, R26, R27: value 220 -> 1K
- R28, R29: value 220 -> 10K
- R35: value 22.1K -> 10K
- R36: value 47.5K -> 10K
- R39: value 11K -> 1K
- R40: value 10 -> 10K
- U3: value ESP32-S3-MINI-1U -> ESP32-S2-MINI-2U-N4; footprint RF_Module:ESP32-S2-MINI-1U -> ESP32_S2_MINI_2U_N4:XCVR_ESP32-S2-MINI-2U-N4
- U4: value 24C02Cx-x-SN -> CP2102N-Axx-xQFN28; footprint Package_DIP:DIP-8_W7.62mm_Socket -> Package_DFN_QFN:QFN-28-1EP_5x5mm_P0.5mm_EP3.35x3.35mm
- U5: value 24C02Cx-x-SN -> ADS1015IDGS; footprint Package_DIP:DIP-8_W7.62mm_Socket -> Package_SO:TSSOP-10_3x3mm_P0.5mm
- U6: value CP2102N-Axx-xQFN28 -> 24C02Cx-x-SN; footprint Package_DFN_QFN:QFN-28-1EP_5x5mm_P0.5mm_EP3.35x3.35mm -> Package_SO:SOIC-8_3.9x4.9mm_P1.27mm
- U7: value LM7171xIM -> 24C02Cx-x-SN
- moved D5 457.6 mm to (519.0, 285.0)
- moved U4 341.1 mm to (503.8, 262.5)
- moved D9 329.9 mm to (138.9, 133.2)
- moved D12 328.1 mm to (85.1, 183.2)
- moved D13 322.9 mm to (453.1, 164.5)
- moved C15 304.9 mm to (493.5, 278.1), turned to 0 degrees
- moved U7 303.6 mm to (493.3, 91.3)
- moved D4 296.1 mm to (499.2, 301.0), turned to 0 degrees
- moved J12 273.2 mm to (507.7, 298.4)
- moved D7 259.0 mm to (512.1, 261.4)
- moved U6 256.8 mm to (501.4, 67.9)
- moved C14 252.4 mm to (493.5, 275.0), turned to 0 degrees
- moved C13 234.8 mm to (493.5, 271.9), turned to 0 degrees
- moved J1 234.7 mm to (335.5, 164.0)
- moved D2 206.1 mm to (249.8, 64.2)
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Connections:
- C10 pad 1: /Chip_PU -> Chip_PU
- C14 pad 1: Net-(U6-VBUS) -> Net-(U4-VBUS)
- C15 pad 1: Net-(C15-Pad1) -> +3.3V
- C15 pad 2: Net-(C15-Pad2) -> GND
- C16 pad 1: +3.3V -> +5V
- C17 pad 1: Net-(C15-Pad1) -> VDDA
- C17 pad 2: /Speaker -> GND
- C2 pad 1: VAA -> +5V
- C5 pad 1: +5V -> +3.3V
- C6 pad 1: +3.3V -> VAA
- D10 pad 1: GND -> Net-(D10-DO)
- D10 pad 2: VBUS -> GND
- D11 pad 1: +5V -> Net-(D11-DO)
- D11 pad 2: VBUS -> GND
- D12 pad 4: Net-(D12-DI) -> Net-(D10-DO)
- D13 pad 1: /Backlight Strip -> Net-(D13-DO)
- D13 pad 4: Net-(D12-DO) -> Net-(D11-DO)
- D14 pad 1: /Out to Power Switch -> Net-(D14-DO)
- D14 pad 2: Net-(D14-A) -> GND
- D15 pad 1: /Out to Power Switch -> Backlight_Strip
- D2 pad 1: Net-(D2-DO) -> Net-(D2-K)
- D2 pad 2: GND -> Net-(D2-A)
- D3 pad 1: Net-(D3-K) -> Net-(D2-K)
- D3 pad 2: Net-(D3-A) -> Power_Off
- D4 pad 1: Net-(D3-K) -> GND
- D4 pad 2: /Power Off -> /USB/USBDP
- D5 pad 1: Net-(D5-DO) -> GND
- D5 pad 2: GND -> /USB/USBDN
- D6 pad 1: Net-(D6-DO) -> GND
- D6 pad 2: GND -> VBUS
- D7 pad 1: GND -> +5V
- D7 pad 2: /USBDP -> VBUS
- D8 pad 1: GND -> Net-(D11-DI)
- D8 pad 2: /USBDN -> GND
- D9 pad 1: Net-(D12-DI) -> Net-(D10-DI)
- D9 pad 4: Net-(D6-DO) -> LED_Data_Out
- J1 pad 2: +5V -> Backlight_Strip
- J1 pad 3: /Servo 1 -> +5V
- J10 pad 2: +5V -> +3.3V
- J10 pad 3: /CL -> CL
- J10 pad 4: /DA -> DA
- J10 pad 5: /CS3 -> CS1
- J10 pad 6: /DC -> DC
- J11 pad 2: +5V -> +3.3V
- J11 pad 3: /Servo 5 -> CL
- J2 pad 2: +5V -> Speaker
- J3 pad 3: /CL -> Servo_1
- J4 pad 3: /Servo 2 -> Servo_2
- J5 pad 1: /Oil In -> GND
- J5 pad 2: /Fuel In -> +5V
- J5 pad 3: /Batt In -> Servo_3
- J6 pad 2: +5V -> SCL
- J6 pad 3: /Servo 3 -> SDA
- J7 pad 1: /Brake In -> GND
- J7 pad 2: /Right Turn In -> +5V
- J7 pad 3: /Left Turn In -> Servo_4
- J8 pad 3: /Servo 4 -> Servo_5
- J9 pad 2: +BATT -> +5V
- J9 pad 3: +VDC -> Servo_6
- Q1 pad 1: /Speed In -> VAA
- Q1 pad 2: +3.3V -> Net-(D2-K)
- Q1 pad 3: /Speed Adjusted -> +BATT
- Q10 pad 1: /Chip_PU -> Net-(Q10-C)
- Q10 pad 3: /RTS -> GND
- Q11 pad 1: /GPIO0 -> Tach_Adjusted
- Q11 pad 3: /DTR -> GND
- Q2 pad 1: /Headlights High In -> Net-(Q2-C)
- Q2 pad 2: +3.3V -> Net-(Q2-B)
- Q2 pad 3: /Headlights High Adjusted -> GND
- Q3 pad 1: /Echo In -> Net-(Q3-C)
- Q3 pad 2: +3.3V -> Net-(Q3-B)
- Q3 pad 3: /Echo Adjusted -> GND
- Q4 pad 1: /Brake In -> Net-(Q4-C)
- Q4 pad 2: +3.3V -> Net-(Q4-B)
- Q4 pad 3: /Brake Adjusted -> GND
- Q5 pad 1: /Tach In -> Speed_Adjusted
- Q5 pad 2: +3.3V -> Net-(Q5-B)
- Q5 pad 3: /Tach Adjusted -> GND
- Q6 pad 1: /Left Turn In -> Headlights_High_Adjusted
- Q6 pad 2: +3.3V -> Net-(Q6-B)
- Q6 pad 3: /Left Turn Adjusted -> GND
- Q7 pad 1: /Headlights Low In -> Brake_Adjusted
- Q7 pad 2: +3.3V -> Net-(Q7-B)
- Q7 pad 3: /Headlights Low Adjusted -> GND
- Q8 pad 1: /Right Turn In -> Net-(Q8-C)
- Q8 pad 2: +3.3V -> Net-(Q8-B)
- Q8 pad 3: /Right Turn Adjusted -> GND
- Q9 pad 1: VAA -> Net-(Q9-C)
- Q9 pad 2: Net-(D3-K) -> Net-(Q9-B)
- Q9 pad 3: /Out to Power Switch -> GND
- R1 pad 1: +3.3V -> Net-(D2-A)
- R1 pad 2: /Speed Adjusted -> GND
- R10 pad 1: +5V -> Net-(U3-IO14)
- R10 pad 2: /Brake In -> Servo_5
- R11 pad 1: +5V -> Net-(U3-IO15)
- R11 pad 2: /Tach In -> Servo_6
- R12 pad 1: +5V -> +3.3V
- R12 pad 2: /Left Turn In -> CS0
- R13 pad 1: +3.3V -> Speed_In
- R13 pad 2: /Headlights Low Adjusted -> Net-(Q2-B)
- R14 pad 1: +3.3V -> Headlights_High_In
- R14 pad 2: /Right Turn Adjusted -> Net-(Q3-B)
- R15 pad 1: +5V -> Brake_In
- R15 pad 2: /Headlights Low In -> Net-(Q4-B)
- R16 pad 1: +5V -> Net-(Q2-C)
- R16 pad 2: /Right Turn In -> VAA
- R17 pad 1: /Trip Reset -> Net-(Q3-C)
- R17 pad 2: GND -> VAA
- R18 pad 1: Net-(D3-A) -> Net-(Q4-C)
- R18 pad 2: GND -> VAA
- R19 pad 1: +3.3V -> Net-(Q2-C)
- R19 pad 2: /Chip_PU -> Net-(Q5-B)
- R2 pad 2: /Headlights High Adjusted -> Chip_PU
- R20 pad 1: Net-(U3-IO17) -> Net-(Q3-C)
- R20 pad 2: /Servo 1 -> Net-(Q6-B)
- R21 pad 1: Net-(U3-IO18) -> Net-(Q4-C)
- R21 pad 2: /Servo 2 -> Net-(Q7-B)
- R22 pad 1: GND -> Speed_Adjusted
- R22 pad 2: Net-(U4-A0) -> +3.3V
- R23 pad 1: GND -> Headlights_High_Adjusted
- R23 pad 2: Net-(U4-A1) -> +3.3V
- R24 pad 1: GND -> Brake_Adjusted
- R24 pad 2: Net-(U4-A2) -> +3.3V
- R25 pad 1: +5V -> Tach_In
- R25 pad 2: /SDA -> Net-(Q8-B)
- R26 pad 1: Net-(U3-IO21) -> Left_Turn_In
- R26 pad 2: /Servo 3 -> Net-(Q9-B)
- R27 pad 1: Net-(U3-IO33) -> Hazard_In
- R27 pad 2: /Servo 4 -> Net-(Q10-B)
- R28 pad 1: Net-(U3-IO34) -> Net-(Q8-C)
- R28 pad 2: /Servo 5 -> VAA
- R29 pad 1: Net-(U3-IO35) -> Net-(Q9-C)
- R29 pad 2: /Servo 6 -> VAA
- R3 pad 2: /Echo Adjusted -> SCL
- R30 pad 1: /DTR -> Net-(Q10-C)
- R30 pad 2: Net-(Q10-B) -> VAA
- R31 pad 1: /RTS -> Net-(Q8-C)
- R32 pad 1: GND -> Net-(Q9-C)
- R32 pad 2: +5V -> Net-(Q12-B)
- R33 pad 1: GND -> Net-(Q10-C)
- R33 pad 2: Net-(U5-A1) -> Net-(Q13-B)
- R34 pad 1: GND -> Tach_Adjusted
- R34 pad 2: Net-(U5-A2) -> +3.3V
- R35 pad 1: Net-(U6-VBUS) -> Left_Turn_Adjusted
- R35 pad 2: VBUS -> +3.3V
- R36 pad 1: Net-(U6-VBUS) -> Hazard_Adjusted
- R36 pad 2: GND -> +3.3V
- R37 pad 1: Net-(U6-~{RST}) -> Headlights_Low_In
- R37 pad 2: GND -> Net-(Q14-B)
- R38 pad 1: +5V -> Right_Turn_In
- R38 pad 2: /SDA -> Net-(Q15-B)
- R39 pad 1: Net-(U6-~{SUSPEND}) -> Echo_In
- R39 pad 2: GND -> Net-(Q16-B)
- R4 pad 1: +5V -> +3.3V
- R4 pad 2: /Speed In -> SDA
- R40 pad 1: Net-(C15-Pad2) -> Net-(Q14-C)
- R40 pad 2: GND -> VAA
- R5 pad 1: +5V -> +3.3V
- R5 pad 2: /Headlights High In -> CS1
- R6 pad 1: +5V -> Net-(U3-IO10)
- R6 pad 2: /Echo In -> Servo_1
- R7 pad 1: +3.3V -> Net-(U3-IO11)
- R7 pad 2: /Brake Adjusted -> Servo_2
- R8 pad 1: +3.3V -> Net-(U3-IO12)
- R8 pad 2: /Tach Adjusted -> Servo_3
- R9 pad 1: +3.3V -> Net-(U3-IO13)
- R9 pad 2: /Left Turn Adjusted -> Servo_4
- SW1 pad 2: /Trip Reset -> Trip_Reset
- U2 pad 2: Net-(D3-A) -> Net-(D2-A)
- U2 pad 3: /Ignition Sensor -> Ignition_Sensor
- U3 pad 10: /Oil In -> unconnected-(U3-IO6-Pad10)
- U3 pad 11: /Trip Reset -> Trip_Reset
- U3 pad 12: /Headlights Low Adjusted -> SDA
- U3 pad 13: /Headlights High Adjusted -> SCL
- U3 pad 14: /Left Turn Adjusted -> Net-(U3-IO10)
- U3 pad 15: /Right Turn Adjusted -> Net-(U3-IO11)
- U3 pad 16: /Brake Adjusted -> Net-(U3-IO12)
- U3 pad 17: /Ignition Sensor -> Net-(U3-IO13)
- U3 pad 18: /Power Off -> Net-(U3-IO14)
- U3 pad 19: /Echo Adjusted -> Net-(U3-IO15)
- U3 pad 20: /Trigger -> Trigger
- U3 pad 21: Net-(U3-IO17) -> Echo_Adjusted
- U3 pad 22: Net-(U3-IO18) -> Left_Turn_Adjusted
- U3 pad 25: Net-(U3-IO21) -> Right_Turn_Adjusted
- U3 pad 26: /CS1 -> unconnected-(U3-IO26-Pad26)
- U3 pad 27: /CS2 -> unconnected-(U3-NC-Pad27)
- U3 pad 28: Net-(U3-IO33) -> Brake_Adjusted
- U3 pad 29: Net-(U3-IO34) -> CS0
- U3 pad 30: /CS3 -> GND
- U3 pad 31: Net-(U3-IO35) -> DA
- U3 pad 32: /LED Data Out -> CL
- U3 pad 33: /SDA -> DC
- U3 pad 34: /SCL -> Headlights_High_Adjusted
- U3 pad 35: /DA -> Ignition_Sensor
- U3 pad 36: /CL -> Power_Off
- U3 pad 37: /DC -> LED_Data_Out
- U3 pad 38: /BL -> Sound_out
- U3 pad 39: /U0TXD -> U0TXD
- U3 pad 4: /GPIO0 -> GPIO0
- U3 pad 40: /U0RXT -> U0RXT
- U3 pad 41: /Sound out -> unconnected-(U3-IO45-Pad41)
- U3 pad 45: /Chip_PU -> Chip_PU
- U3 pad 5: /Tach Adjusted -> Tach_Adjusted
- U3 pad 6: /Speed Adjusted -> Speed_Adjusted
- U3 pad 7: /Temp In -> Headlights_Low_Adjusted
- U3 pad 8: /Batt In -> CS1
- U3 pad 9: /Fuel In -> Hazard_Adjusted
- U4 pad 1: Net-(U4-A0) -> unconnected-(U4-~{DCD}-Pad1)
- U4 pad 2: Net-(U4-A1) -> unconnected-(U4-~{RI}/CLK-Pad2)
- U4 pad 3: Net-(U4-A2) -> GND
- U4 pad 4: GND -> /USB/USBDP
- U4 pad 5: /SDA -> /USB/USBDN
- U4 pad 6: /SCL -> +3.3V
- U4 pad 7: GND -> +3.3V
- U4 pad 8: +5V -> Net-(U4-VBUS)
- U5 pad 1: +5V -> GND
- U5 pad 2: Net-(U5-A1) -> unconnected-(U5-ALERT/RDY-Pad2)
- U5 pad 3: Net-(U5-A2) -> GND
- U5 pad 4: GND -> Temp_In
- U5 pad 5: /SDA -> Batt_In
- U5 pad 6: /SCL -> Fuel_In
- U5 pad 7: GND -> Oil_In
- U5 pad 8: +5V -> VDDA
- U6 pad 1: unconnected-(U6-~{DCD}-Pad1) -> Net-(U6-A0)
- U6 pad 2: unconnected-(U6-~{RI}/CLK-Pad2) -> Net-(U6-A1)
- U6 pad 3: GND -> Net-(U6-A2)
- U6 pad 4: /USBDP -> GND
- U6 pad 5: /USBDN -> SDA
- U6 pad 6: +3.3V -> SCL
- U6 pad 7: +3.3V -> GND
- U6 pad 8: Net-(U6-VBUS) -> +3.3V
- U7 pad 1: unconnected-(U7-NC-Pad1) -> +3.3V
- U7 pad 2: GND -> Net-(U7-A1)
- U7 pad 3: /Sound out -> Net-(U7-A2)
- U7 pad 5: unconnected-(U7-NC-Pad5) -> SDA
- U7 pad 6: Net-(C15-Pad1) -> SCL
- U7 pad 7: VAA -> GND
- U7 pad 8: unconnected-(U7-NC-Pad8) -> +3.3V
Routing:
- net GND: track 0.00 -> 46.4 mm, vias 0 -> 50
- net +3.3V: track 0.00 -> 38.8 mm
- net +5V: track 0.00 -> 31.8 mm
- net Net-(D1-K): track 0.00 -> 29.2 mm
- net VAA: track 0.00 -> 18.9 mm
- net Net-(Q14-C): track 0.00 -> 17.3 mm
- net Net-(Q2-C): track 0.00 -> 17.3 mm
- net Net-(Q9-C): track 0.00 -> 17.2 mm
- net Net-(Q10-C): track 0.00 -> 17.2 mm
- net Net-(Q3-C): track 0.00 -> 17.2 mm
- net Net-(Q15-C): track 0.00 -> 17.2 mm
- net Net-(Q16-C): track 0.00 -> 17.2 mm
- net Net-(Q4-C): track 0.00 -> 17.1 mm
- net Net-(Q8-C): track 0.00 -> 17.1 mm
- net Net-(U3-IO15): track 0.00 -> 13.1 mm
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- added copper zone on B.Cu, net GND
Other:
- outline, holes or cut-outs redrawn

Commit message: Update
Parts:
- removed FB2: FerriteBead_Small, Inductor_THT:L_Axial_L5.0mm_D3.6mm_P10.00mm_Horizontal_Murata_BL01RN1A2A2
- moved C1 165.5 mm to (343.0, 127.2)
- moved C2 165.5 mm to (337.2, 138.5)
- moved C3 165.5 mm to (331.5, 127.2)
- moved C4 165.5 mm to (337.2, 127.3)
- moved C5 165.5 mm to (325.8, 138.5)
- moved C6 165.5 mm to (346.8, 125.0)
- moved C7 165.5 mm to (347.0, 132.2)
- moved C9 165.5 mm to (343.0, 138.5)
- moved D1 165.5 mm to (350.3, 135.0)
- moved IC1 165.5 mm to (348.1, 128.6)
- moved L1 165.5 mm to (355.2, 127.0)
- moved U1 165.5 mm to (330.8, 141.8)
- moved C8 165.5 mm to (348.8, 138.3)
- moved C18 149.9 mm to (227.2, 132.0), turned to 180 degrees
- moved C17 145.7 mm to (232.2, 132.0), turned to 180 degrees
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Connections:
- J6 pad 10: +BATT -> +VDC
- J6 pad 11: +VDC -> Batt_In
- J6 pad 12: Brake_In -> Temp_In
- J6 pad 13: Hazard_In -> Fuel_In
- J6 pad 14: Right_Turn_In -> Oil_In
- J6 pad 15: Left_Turn_In -> Tach_In
- J6 pad 16: Headlights_High_In -> Speed_In
- J6 pad 18: Oil_In -> Hazard_In
- J6 pad 19: Fuel_In -> Echo_In
- J6 pad 20: Batt_In -> Left_Turn_In
- J6 pad 21: Temp_In -> Right_Turn_In
- J6 pad 22: Tach_In -> Brake_In
- J6 pad 23: Speed_In -> Headlights_High_In
- J6 pad 6: Echo_In -> Trigger
- J6 pad 7: Trigger -> +5V
- J6 pad 8: +5V -> GND
- J6 pad 9: GND -> +BATT
- U3 pad 21: Echo_Adjusted -> Power_Off
- U3 pad 22: Left_Turn_Adjusted -> Ignition_Sensor
- U3 pad 25: Right_Turn_Adjusted -> DC
- U3 pad 28: Brake_Adjusted -> CS0
- U3 pad 29: CS0 -> Headlights_High_Adjusted
- U3 pad 31: DA -> Brake_Adjusted
- U3 pad 32: CL -> Right_Turn_Adjusted
- U3 pad 33: DC -> Left_Turn_Adjusted
- U3 pad 34: Headlights_High_Adjusted -> Echo_Adjusted
- U3 pad 35: Ignition_Sensor -> Hazard_Adjusted
- U3 pad 36: Power_Off -> Headlights_Low_Adjusted
- U3 pad 37: LED_Data_Out -> Speed_Adjusted
- U3 pad 38: Sound_out -> Tach_Adjusted
- U3 pad 5: Tach_Adjusted -> Sound_out
- U3 pad 6: Speed_Adjusted -> LED_Data_Out
- U3 pad 7: Headlights_Low_Adjusted -> DA
- U3 pad 9: Hazard_Adjusted -> CL
Routing:
- net Net-(D11-DI): track 0.00 -> 195.3 mm
- net Net-(D12-DO): track 0.00 -> 190.2 mm
- net Tach_Adjusted: track 4.32 -> 119.3 mm, vias 1 -> 0
- net Speed_Adjusted: track 4.45 -> 105.2 mm, vias 1 -> 0
- net Tach_In: track 0.00 -> 88.3 mm
- net Headlights_Low_Adjusted: track 4.27 -> 91.1 mm, vias 1 -> 0
- net Backlight_Strip: track 0.00 -> 78.3 mm
- net Hazard_Adjusted: track 4.14 -> 79.8 mm, vias 1 -> 0
- net Speed_In: track 0.00 -> 74.8 mm
- net Net-(D13-DO): track 0.00 -> 73.0 mm
- net Echo_Adjusted: track 4.09 -> 67.5 mm, vias 1 -> 0
- net Headlights_Low_In: track 0.00 -> 61.6 mm
- net Batt_In: track 0.00 -> 61.0 mm
- net Temp_In: track 0.00 -> 58.4 mm
- net Fuel_In: track 0.00 -> 51.8 mm
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
Commit message: update
Parts:
- moved J3 15.6 mm to (103.2, 165.4)
- moved J4 15.5 mm to (103.0, 181.0)
Routing:
- net +3.3V: track 52.8 -> 354.0 mm, vias 0 -> 8
- net VAA: track 55.4 -> 187.1 mm
- net SDA: track 11.7 -> 125.4 mm, vias 0 -> 4
- net SCL: track 9.65 -> 121.1 mm, vias 0 -> 4
- net GND: track 48.9 -> 69.9 mm, vias 52 -> 48
- net Servo_3: track 0.00 -> 13.9 mm
- net Servo_2: track 0.00 -> 12.9 mm
- net Servo_1: track 0.00 -> 9.77 mm
- net VDDA: track 16.7 -> 18.2 mm
Other:
- copper layers 2 -> 4

Commit message: update
Parts:
- SW2, SW3: moved to B.Cu
- U6, U7, U8: footprint Package_SO:SOIC-8_3.9x4.9mm_P1.27mm -> Package_DIP:DIP-8_W7.62mm
- moved Q20 394.6 mm to (134.5, 172.0), turned to 180 degrees
- moved Q21 390.8 mm to (140.0, 171.9), turned to 180 degrees
- moved D5 384.1 mm to (152.0, 171.7), turned to 180 degrees
- moved J12 382.8 mm to (145.5, 174.6)
- moved D6 381.3 mm to (155.6, 176.9), turned to 90 degrees
- moved D4 377.1 mm to (145.0, 171.7)
- moved R54 375.3 mm to (150.1, 162.1), turned to 180 degrees
- moved R50 375.0 mm to (143.9, 165.3), turned to 180 degrees
- moved R53 374.9 mm to (150.1, 159.1), turned to 180 degrees
- moved R49 372.9 mm to (143.9, 168.3), turned to 180 degrees
- moved R51 369.8 mm to (152.8, 158.8), turned to -90 degrees
- moved U4 368.3 mm to (148.2, 166.8), turned to 90 degrees
- moved R52 368.3 mm to (155.8, 158.8), turned to -90 degrees
- moved D7 365.0 mm to (159.0, 169.0), turned to -90 degrees
- moved C14 354.7 mm to (158.4, 158.8), turned to -90 degrees
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Connections:
- net /USB/USBDN renamed /USB/USB_D_N
- net /USB/USBDP renamed /USB/USB_D_P
- U3 pad 11: Trip_Reset -> CL
- U3 pad 25: DC -> Trip_Reset
- U3 pad 28: CS0 -> Sound_out
- U3 pad 5: Sound_out -> LED_Data_Out
- U3 pad 6: LED_Data_Out -> DC
- U3 pad 9: CL -> CS0
Routing:
- net +5V: track 35.7 -> 889.8 mm, vias 0 -> 11
- net DC: track 0.00 -> 297.0 mm, vias 0 -> 4
- net DA: track 0.00 -> 296.2 mm, vias 0 -> 4
- net CS1: track 0.00 -> 289.5 mm, vias 0 -> 5
- net CL: track 0.00 -> 283.8 mm, vias 0 -> 4
- net Servo_5: track 0.00 -> 242.3 mm
- net Servo_6: track 0.00 -> 236.6 mm
- net +3.3V: track 354.0 -> 578.4 mm, vias 8 -> 17
- net Chip_PU: track 0.00 -> 192.9 mm, vias 0 -> 6
- net Servo_4: track 0.00 -> 157.3 mm
- net Trip_Reset: track 0.00 -> 153.1 mm, vias 0 -> 4
- net GPIO0: track 0.00 -> 149.9 mm, vias 0 -> 7
- net CS0: track 0.97 -> 137.1 mm, vias 1 -> 6
- net Ignition_Sensor: track 0.00 -> 134.1 mm, vias 0 -> 5
- net U0RXT: track 0.00 -> 126.7 mm, vias 0 -> 6
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Other:
- outline, holes or cut-outs redrawn
- copper layers 4 -> 2

Commit message: update
Connections:
- net Servo_1 renamed Oil_Servo
- net Servo_2 renamed Fuel_Servo
- net Servo_3 renamed Speed_Servo
- net Servo_4 renamed Tach_Servo
- net Servo_5 renamed Temp_Servo
- net Servo_6 renamed Batt_Servo
