File: Instrument Panel Final.kicad_pcb (KiCad board)
At the start: 2 copper layers, 401.2 x 87.2 mm, 145 parts, among them IC1 LM2678SD-5.0_NOPB, J1 Conn_01x03_Socket, J10 Conn_01x06_Socket, J11 Conn_01x06_Socket, J12 USB_C_Receptacle_USB2.0_14P, J2 Conn_01x02_Socket, J3 Conn_01x03_Socket, J4 Conn_01x03_Socket, J5 Conn_01x03_Socket, J6 Conn_01x23_Socket, J7 Conn_01x03_Socket, J8 Conn_01x03_Socket, J9 Conn_01x03_Socket, Q1 2N7000, Q10 NPN, Q11 NPN, Q12 NPN, Q13 NPN, Q14 NPN, Q15 NPN, Q16 NPN, Q17 NPN, Q18 NPN, Q19 NPN, Q2 NPN, Q20 NPN, Q21 NPN, Q3 NPN, Q4 NPN, Q5 NPN, Q6 NPN, Q7 NPN, Q8 NPN, Q9 NPN, SW1 SW_Push, SW2 SW_Push, SW3 SW_Push, U1 UA78M33QDCYRQ1, U2 SFH617A-1, U3 ESP32-S2-MINI-2U-N4, U4 CP2102N-Axx-xQFN28, U5 ADS1015IDGS, U6 24C02Cx-x-SN, U7 24C02Cx-x-SN, U8 LM7171xIM

Commit message: update
Parts:
- added D17: D_Schottky, Diode_SMD:Vishay_SMPA, F.Cu at (288.8, 136.8)
- added D18: SMF18A, Diode_SMD:D_SMF, F.Cu at (288.1, 139.6)
- added D19: 1N914, Diode_THT:D_DO-35_SOD27_P7.62mm_Horizontal, F.Cu at (304.8, 138.2)
- added D20: SMF18A, Diode_SMD:D_SMF, F.Cu at (303.6, 140.6)
- added F1: Polyfuse, Fuse:Fuse_BelFuse_0ZRE0005FF_L8.3mm_W3.8mm, F.Cu at (282.8, 139.1)
- added F2: Polyfuse, Fuse:Fuse_1210_3225Metric, F.Cu at (294.4, 139.2)
- R1: value 150 -> 470
Connections:
- Q1 pad 3: +BATT -> /Power/Constant Power
- U2 pad 1: +VDC -> /Power/Switched Power
Routing:
- net /Power/Switched Power: track 0.00 -> 40.4 mm, vias 0 -> 1
- net /Power/Constant Power: track 0.00 -> 24.3 mm, vias 0 -> 1
- net +BATT: track 29.4 -> 10.7 mm
- net +VDC: track 43.4 -> 32.1 mm, vias 0 -> 1
- net GND: track 92.2 -> 102.5 mm, vias 54 -> 109
- net Net-(D17-A): track 0.00 -> 4.95 mm
- net Net-(D19-A): track 0.00 -> 3.77 mm
- net VBUS: track 27.2 -> 28.5 mm
- added copper zone on F.Cu, net GND

Commit message: update
Parts:
- removed J3, J4, J5, J7, J8, J9: Conn_01x03_Socket, Connector_Hirose:Hirose_DF13-03P-1.25DSA_1x03_P1.25mm_Vertical
- removed R10, R11, R6, R7, R8, R9: 220, Resistor_THT:R_Axial_DIN0207_L6.3mm_D2.5mm_P10.16mm_Horizontal
- added C21: 100n, Capacitor_THT:C_Disc_D3.0mm_W1.6mm_P2.50mm, F.Cu at (372.7, 163.4)
- added C22: 100n, Capacitor_THT:C_Disc_D3.0mm_W1.6mm_P2.50mm, F.Cu at (372.6, 148.8)
- added C23: 100n, Capacitor_THT:C_Disc_D3.0mm_W1.6mm_P2.50mm, F.Cu at (372.6, 134.4)
- added C24: 100n, Capacitor_THT:C_Disc_D3.0mm_W1.6mm_P2.50mm, F.Cu at (246.6, 164.1)
- added C25: 100n, Capacitor_THT:C_Disc_D3.0mm_W1.6mm_P2.50mm, F.Cu at (264.3, 176.3)
- added C26: 100n, Capacitor_THT:C_Disc_D3.0mm_W1.6mm_P2.50mm, F.Cu at (270.4, 164.0)
- added C27: 100n, Capacitor_THT:C_Disc_D3.0mm_W1.6mm_P2.50mm, F.Cu at (288.2, 176.2)
- added C28: 100n, Capacitor_THT:C_Disc_D3.0mm_W1.6mm_P2.50mm, F.Cu at (445.2, 159.2)
- added C29: 100n, Capacitor_THT:C_Disc_D3.0mm_W1.6mm_P2.50mm, F.Cu at (427.7, 182.0)
- added C30: 100n, Capacitor_THT:C_Disc_D3.0mm_W1.6mm_P2.50mm, F.Cu at (118.0, 190.2)
- added C31: 100n, Capacitor_THT:C_Disc_D3.0mm_W1.6mm_P2.50mm, F.Cu at (100.0, 178.0)
- added C32: 100n, Capacitor_THT:C_Disc_D3.0mm_W1.6mm_P2.50mm, F.Cu at (99.9, 147.7)
- added C33: 100n, Capacitor_THT:C_Disc_D3.0mm_W1.6mm_P2.50mm, F.Cu at (117.7, 159.7)
- added C34: 100n, Capacitor_THT:C_Disc_D3.0mm_W1.6mm_P2.50mm, F.Cu at (445.4, 194.0)
- added C35: 100n, Capacitor_THT:C_Disc_D3.0mm_W1.6mm_P2.50mm, F.Cu at (427.3, 147.2)
- added J13: Conn_01x04_Socket, Connector_Hirose:Hirose_DF13-04P-1.25DSA_1x04_P1.25mm_Vertical, F.Cu at (434.4, 180.9)
- added J14: Conn_01x04_Socket, Connector_Hirose:Hirose_DF13-04P-1.25DSA_1x04_P1.25mm_Vertical, F.Cu at (438.1, 160.2)
- added J15: Conn_01x04_Socket, Connector_Hirose:Hirose_DF13-04P-1.25DSA_1x04_P1.25mm_Vertical, F.Cu at (281.3, 177.2)
- added J16: Conn_01x04_Socket, Connector_Hirose:Hirose_DF13-04P-1.25DSA_1x04_P1.25mm_Vertical, F.Cu at (257.4, 177.3)
- added J17: Conn_01x04_Socket, Connector_Hirose:Hirose_DF13-04P-1.25DSA_1x04_P1.25mm_Vertical, F.Cu at (110.9, 160.6)
- added J18: Conn_01x04_Socket, Connector_Hirose:Hirose_DF13-04P-1.25DSA_1x04_P1.25mm_Vertical, F.Cu at (107.2, 177.0)
- added R63: 10K, Resistor_THT:R_Axial_DIN0207_L6.3mm_D2.5mm_P10.16mm_Horizontal, F.Cu at (389.4, 162.8)
- added R64: 10K, Resistor_THT:R_Axial_DIN0207_L6.3mm_D2.5mm_P10.16mm_Horizontal, F.Cu at (389.0, 148.4)
- added R65: 10K, Resistor_THT:R_Axial_DIN0207_L6.3mm_D2.5mm_P10.16mm_Horizontal, F.Cu at (388.9, 134.0)
- added U10: 74HC595, Package_DIP:DIP-16_W7.62mm, F.Cu at (372.5, 158.6)
- added U11: 74HC595, Package_DIP:DIP-16_W7.62mm, F.Cu at (372.4, 144.2)
- added U12: L293D, Package_DIP:DIP-16_W7.62mm, F.Cu at (100.0, 157.4)
- added U13: L293D, Package_DIP:DIP-16_W7.62mm, F.Cu at (117.9, 180.3)
- added U14: L293D, Package_DIP:DIP-16_W7.62mm, F.Cu at (270.5, 173.9)
- added U15: L293D, Package_DIP:DIP-16_W7.62mm, F.Cu at (246.5, 174.0)
- added U16: L293D, Package_DIP:DIP-16_W7.62mm, F.Cu at (445.4, 184.2)
- added U17: L293D, Package_DIP:DIP-16_W7.62mm, F.Cu at (427.2, 157.0)
- added U9: 74HC595, Package_DIP:DIP-16_W7.62mm, F.Cu at (372.7, 173.2)
Routing:
- net Net-(U13-3A): track 0.00 -> 345.5 mm, vias 0 -> 14
- net Net-(U13-2A): track 0.00 -> 341.9 mm, vias 0 -> 15
- net Net-(U13-4A): track 0.00 -> 336.3 mm, vias 0 -> 14
- net +5V: track 889.8 -> 1217.7 mm, vias 11 -> 10
- net Net-(U13-1A): track 0.00 -> 327.2 mm, vias 0 -> 14
- net Net-(U12-4A): track 0.00 -> 316.4 mm, vias 0 -> 12
- net Net-(U12-1A): track 0.00 -> 314.5 mm, vias 0 -> 13
- net Net-(U12-3A): track 0.00 -> 302.4 mm, vias 0 -> 12
- net Net-(U12-2A): track 0.00 -> 295.1 mm, vias 0 -> 11
- net Temp_Servo: track 242.3 -> 0.00 mm
- net Batt_Servo: track 236.6 -> 0.00 mm
- net Tach_Servo: track 157.3 -> 0.00 mm
- net Net-(U10-QH): track 0.00 -> 152.3 mm, vias 0 -> 4
- net Net-(U10-QE): track 0.00 -> 148.0 mm, vias 0 -> 5
- net Net-(U10-QG): track 0.00 -> 137.8 mm, vias 0 -> 5
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
Commit message: update
Parts:
- removed D2, D3: D, Diode_THT:D_A-405_P7.62mm_Horizontal
- removed Q1: 2N7000, Package_TO_SOT_THT:TO-92_Inline
- removed R1: 470, Resistor_THT:R_Axial_DIN0207_L6.3mm_D2.5mm_P10.16mm_Horizontal
- removed U2: SFH617A-1, Package_DIP:DIP-4_W7.62mm
- added D21: D, Diode_THT:D_A-405_P7.62mm_Horizontal, F.Cu at (317.1, 140.1)
- added D22: D, Diode_THT:D_A-405_P7.62mm_Horizontal, F.Cu at (317.1, 135.9)
- added Q22: PMOS, Package_TO_SOT_THT:TO-220-3_Vertical, F.Cu at (320.5, 130.6)
- added Q23: NMOS, Package_TO_SOT_THT:TO-220-3_Vertical, F.Cu at (309.7, 130.6)
- added R66: 10k, Resistor_THT:R_Axial_DIN0207_L6.3mm_D2.5mm_P10.16mm_Horizontal, F.Cu at (308.5, 155.3)
- added R67: 10k, Resistor_THT:R_Axial_DIN0207_L6.3mm_D2.5mm_P10.16mm_Horizontal, F.Cu at (311.5, 145.1)
- added R68: 47k, Resistor_THT:R_Axial_DIN0207_L6.3mm_D2.5mm_P10.16mm_Horizontal, F.Cu at (314.6, 145.1)
- added R69: 1k, Resistor_THT:R_Axial_DIN0207_L6.3mm_D2.5mm_P10.16mm_Horizontal, F.Cu at (317.6, 145.1)
- added R70: 1k, Resistor_THT:R_Axial_DIN0207_L6.3mm_D2.5mm_P10.16mm_Horizontal, F.Cu at (320.6, 145.1)
- added R71: 10k, Resistor_THT:R_Axial_DIN0207_L6.3mm_D2.5mm_P10.16mm_Horizontal, F.Cu at (323.7, 155.3)
- added U18: SFH617A-1, Package_DIP:DIP-4_W7.62mm, F.Cu at (321.0, 137.6)
- L1: footprint Inductor_THT:L_Radial_D9.5mm_P5.00mm_Fastron_07HVP -> Inductor_THT:L_Axial_L9.5mm_D4.0mm_P15.24mm_Horizontal_Fastron_SMCC
- moved Q5 18.2 mm to (287.4, 158.4)
- moved Q8 18.2 mm to (304.9, 158.3)
- moved R13 18.2 mm to (290.3, 145.1)
- moved R16 18.2 mm to (293.3, 155.3)
- moved R22 18.2 mm to (287.3, 155.3)
- moved Q15 18.2 mm to (232.5, 158.4)
- moved Q3 18.2 mm to (208.1, 158.4)
- moved Q6 18.2 mm to (202.6, 158.5)
- moved Q7 18.2 mm to (214.7, 158.5)
- moved Q9 18.2 mm to (244.6, 158.4)
- moved R14 18.2 mm to (205.6, 145.2)
- moved R15 18.2 mm to (217.7, 145.2)
- moved R17 18.2 mm to (208.6, 155.4)
- moved R18 18.2 mm to (220.7, 155.4)
- moved R20 18.2 mm to (199.5, 145.2)
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Connections:
- net /Power/Constant Power renamed /USB and Power/Constant Power
- net /Power/Switched Power renamed /USB and Power/Switched Power
- net /USB/DTR renamed /USB and Power/DTR
- net /USB/RTS renamed /USB and Power/RTS
- net /USB/USB_D_N renamed /USB and Power/USB_D_N
- net /USB/USB_D_P renamed /USB and Power/USB_D_P
- net Trip_Reset renamed /Trip Reset
- U3 pad 14: Net-(U3-IO10) -> unconnected-(U3-IO10-Pad14)
- U3 pad 15: Net-(U3-IO11) -> unconnected-(U3-IO11-Pad15)
- U3 pad 16: Net-(U3-IO12) -> unconnected-(U3-IO12-Pad16)
- U3 pad 17: Net-(U3-IO13) -> unconnected-(U3-IO13-Pad17)
- U3 pad 18: Net-(U3-IO14) -> unconnected-(U3-IO14-Pad18)
- U3 pad 19: Net-(U3-IO15) -> CS2
Routing:
- net CS2: track 66.4 -> 265.1 mm, vias 0 -> 10
- net +3.3V: track 586.5 -> 510.7 mm, vias 17 -> 7
- net /Trip Reset: track 152.1 -> 102.0 mm, vias 4 -> 3
- net Backlight_Strip: track 86.4 -> 44.5 mm
- net Net-(Q22-G): track 0.00 -> 40.8 mm
- net /USB and Power/Switched Power: track 40.4 -> 2.50 mm, vias 1 -> 0
- net /USB and Power/Constant Power: track 24.3 -> 61.9 mm, vias 1 -> 0
- net Sound_out: track 39.9 -> 5.43 mm
- net Left_Turn_Adjusted: track 55.4 -> 25.4 mm
- net +5V: track 1217.7 -> 1191.4 mm, vias 10 -> 11
- net Tach_Adjusted: track 119.3 -> 98.3 mm
- net Net-(D21-K): track 0.00 -> 20.2 mm
- net Net-(D21-A): track 0.00 -> 19.2 mm
- net Brake_In: track 37.1 -> 56.2 mm
- net Right_Turn_In: track 23.2 -> 42.0 mm
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