File: Instrument Panel Final.kicad_pcb (KiCad board)
At the start: 2 copper layers, 401.2 x 87.2 mm, 178 parts, among them IC1 LM2678SD-5.0_NOPB, J1 Conn_01x03_Socket, J10 Conn_01x06_Socket, J11 Conn_01x06_Socket, J12 USB_C_Receptacle_USB2.0_14P, J13 Conn_01x04_Socket, J14 Conn_01x04_Socket, J15 Conn_01x04_Socket, J16 Conn_01x04_Socket, J17 Conn_01x04_Socket, J18 Conn_01x04_Socket, J2 Conn_01x02_Socket, J6 Conn_01x23_Socket, Q10 NPN, Q11 NPN, Q12 NPN, Q13 NPN, Q14 NPN, Q15 NPN, Q16 NPN, Q17 NPN, Q18 NPN, Q19 NPN, Q2 NPN, Q20 NPN, Q21 NPN, Q22 PMOS, Q23 NMOS, Q3 NPN, Q4 NPN, Q5 NPN, Q6 NPN, Q7 NPN, Q8 NPN, Q9 NPN, SW1 SW_Push, SW2 SW_Push, SW3 SW_Push, U1 UA78M33QDCYRQ1, U10 74HC595, U11 74HC595, U12 L293D, U13 L293D, U14 L293D, U15 L293D, U16 L293D, U17 L293D, U18 SFH617A-1, U3 ESP32-S2-MINI-2U-N4, U4 CP2102N-Axx-xQFN28, U5 ADS1015IDGS, U6 24C02Cx-x-SN, U7 24C02Cx-x-SN, U8 LM7171xIM, U9 74HC595

Commit message: update
Parts:
- moved C24 1.71 mm to (246.6, 162.4)
- moved C25 1.71 mm to (264.3, 174.6)
- moved J15 1.71 mm to (281.3, 175.5)
- moved U15 1.71 mm to (246.5, 172.3)
- moved C26 1.71 mm to (270.4, 162.3)
- moved C27 1.71 mm to (288.2, 174.5)
- moved J16 1.71 mm to (257.4, 175.6)
- moved U14 1.71 mm to (270.4, 172.2)
- moved D6 0.15 mm to (155.6, 177.1)
- moved Q9 0.10 mm to (244.6, 158.5)
- moved R29 0.08 mm to (245.1, 155.4)
Routing:
- net Net-(U10-QE): track 144.8 -> 93.3 mm, vias 5 -> 4
- net CS1: track 303.3 -> 252.9 mm, vias 5 -> 3
- net CL: track 391.2 -> 341.7 mm, vias 7 -> 8
- net Net-(U10-QH): track 147.8 -> 98.9 mm
- net DA: track 340.8 -> 293.6 mm, vias 6 -> 4
- net DC: track 306.8 -> 260.6 mm, vias 4 -> 2
- net Backlight_Strip: track 44.5 -> 90.4 mm, vias 0 -> 2
- net Sound_out: track 5.43 -> 50.6 mm, vias 0 -> 2
- net +5V: track 1191.4 -> 1150.6 mm
- net Net-(U10-QF): track 133.7 -> 93.8 mm, vias 5 -> 4
- net Net-(U10-QG): track 133.4 -> 96.1 mm, vias 5 -> 4
- net Net-(U10-QA): track 114.9 -> 85.1 mm, vias 5 -> 4
- net /Trip Reset: track 102.0 -> 131.1 mm, vias 3 -> 4
- net Net-(U10-QD): track 114.6 -> 88.5 mm, vias 5 -> 4
- net Ignition_Sensor: track 121.0 -> 146.2 mm, vias 4 -> 5
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Other:
- outline, holes or cut-outs redrawn

Commit message: update
Routing:
- net CS1: track 252.9 -> 304.0 mm
- net CL: track 341.7 -> 392.4 mm
- net Net-(U10-QH): track 98.9 -> 148.8 mm, vias 4 -> 1
- net Net-(U10-QE): track 93.3 -> 141.4 mm, vias 4 -> 3
- net DA: track 293.6 -> 341.7 mm
- net +3.3V: track 511.8 -> 559.7 mm, vias 7 -> 12
- net DC: track 260.6 -> 307.1 mm
- net Net-(U10-QF): track 93.8 -> 130.4 mm, vias 4 -> 2
- net Net-(U10-QG): track 96.1 -> 132.7 mm, vias 4 -> 2
- net Net-(U10-QA): track 85.1 -> 114.7 mm, vias 4 -> 3
- net Net-(U10-QD): track 88.5 -> 113.6 mm, vias 4 -> 2
- net +5V: track 1150.6 -> 1169.2 mm, vias 11 -> 15
- net /Trip Reset: track 131.1 -> 149.4 mm, vias 4 -> 6
- net Net-(U10-QC): track 84.8 -> 98.9 mm, vias 4 -> 2
- net Net-(J16-Pin_3): track 0.38 -> 13.1 mm, vias 0 -> 2
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
Commit message: update
Parts:
- moved D6 12.0 mm to (143.6, 178.2)
- moved J12 2.91 mm to (147.9, 176.2)
Routing:
- net /USB and Power/Switched Power: track 2.50 -> 19.0 mm, vias 0 -> 1
- net GND: track 99.1 -> 88.6 mm, vias 118 -> 114
- net VAA: track 249.3 -> 254.0 mm
- net VBUS: track 28.5 -> 32.1 mm
- net /USB and Power/USB_D_P: track 7.90 -> 10.4 mm, vias 0 -> 1
- net Net-(D12-DO): track 199.5 -> 201.9 mm
- net Brake_Adjusted: track 30.6 -> 29.0 mm
- net /USB and Power/USB_D_N: track 8.01 -> 9.52 mm, vias 0 -> 1
- net DA: track 341.7 -> 340.5 mm
- net +5V: track 1169.2 -> 1170.4 mm, vias 15 -> 17
- net Chip_PU: track 189.8 -> 189.0 mm
- net DC: track 307.1 -> 306.4 mm
- net CL: track 392.4 -> 391.8 mm
- net /USB and Power/Constant Power: track 65.1 -> 65.6 mm
