File: power.kicad_sch (KiCad schematic)
At the start: 18 parts, among them IC1 LM2678SD-5.0_NOPB, Q1 2N7000, U1 UA78M33QDCYRQ1, U2 SFH617A-1

Commit message: update
Parts:
- added D17: D_Schottky, Diode_SMD:Vishay_SMPA, symbol Device:D_Schottky
- added D18, D20: SMF18A, Diode_SMD:D_SMF, symbol Diode:SMF18A
- added D19: 1N914, Diode_THT:D_DO-35_SOD27_P7.62mm_Horizontal, symbol Diode:1N914
- added F1: Polyfuse, Fuse:Fuse_BelFuse_0ZRE0005FF_L8.3mm_W3.8mm, symbol Device:Polyfuse
- added F2: Polyfuse, Fuse:Fuse_1210_3225Metric, symbol Device:Polyfuse
- R1: value 150 -> 470
Connections:
- net +BATT: now also F1.2; no longer Q1.3 (D)
- net +VDC: now also F2.2; no longer U2.1
- net GND: now also D18.2 (A2), D20.2 (A2)
- new net: D17.2 (A), F1.1
- new net: D19.2 (A), F2.1
- new net Constant Power: D17.1 (K), D18.1 (A1), Q1.3 (D)
- new net Switched Power: D19.1 (K), D20.1 (A1), U2.1
Other:
- note added: "0ZRB0400FF1A"
- note added: "B59807A0090A062"
- note added: "Constant power protection"
- note added: "Switched power protection"
- note added: "V8PAM10HM3"
- note removed: "Constant +12 from battery"
- note removed: "Switched +12 from battery"

Commit message: update
Parts:
- added C13, C15: 10u, Capacitor_THT:C_Disc_D3.0mm_W1.6mm_P2.50mm, symbol Device:C
- added C14: 1u, Capacitor_THT:C_Disc_D3.0mm_W1.6mm_P2.50mm, symbol Device:C
- added D4, D5, D6: SMAJ5.0CA, Diode_SMD:D_SMA, symbol Diode:SMAJ5.0CA
- added D7: 1N5819, Diode_THT:D_DO-41_SOD81_P10.16mm_Horizontal, symbol Diode:1N5819
- added J12: USB_C_Receptacle_USB2.0_14P, Connector_USB:USB_C_Receptacle_GCT_USB4085, symbol Connector:USB_C_Receptacle_USB2.0_14P
- added Q20, Q21: NPN, Package_TO_SOT_THT:TO-92_Inline, symbol Simulation_SPICE:NPN
- added R49, R50: 10K, Resistor_THT:R_Axial_DIN0207_L6.3mm_D2.5mm_P10.16mm_Horizontal, symbol Device:R
- added R51: 22.1K, Resistor_THT:R_Axial_DIN0207_L6.3mm_D2.5mm_P10.16mm_Horizontal, symbol Device:R
- added R52: 47.5K, Resistor_THT:R_Axial_DIN0207_L6.3mm_D2.5mm_P10.16mm_Horizontal, symbol Device:R
- added R53: 1K, Resistor_THT:R_Axial_DIN0207_L6.3mm_D2.5mm_P10.16mm_Horizontal, symbol Device:R
- added R54: 11K, Resistor_THT:R_Axial_DIN0207_L6.3mm_D2.5mm_P10.16mm_Horizontal, symbol Device:R
- added U4: CP2102N-Axx-xQFN28, Package_DFN_QFN:QFN-28-1EP_5x5mm_P0.5mm_EP3.35x3.35mm, symbol Interface_USB:CP2102N-Axx-xQFN28
Connections:
- net +3.3V: now also C15.1, U4.6 (VDD), U4.7 (VREGIN)
- net +5V: now also C13.1, D7.1 (K)
- net GND: now also C13.2, C14.2, C15.2, D4.1 (A1), D5.1 (A1), D6.1 (A1), J12.A1 (GND), J12.A12 (GND), J12.B1 (GND), J12.B12 (GND), J12.SH (SHIELD), R52.2, R53.2, R54.2, U4.29 (GND), U4.3 (GND); no longer C3.2
- net VBUS: now also D6.2 (A2), D7.2 (A), J12.A4 (VBUS), J12.A9 (VBUS), J12.B4 (VBUS), J12.B9 (VBUS), R51.2
- new net: R54.1, U4.11 (~{SUSPEND})
- new net: R53.1, U4.9 (~{RST})
- new net: Q21.2 (B), R50.2
- new net: C14.1, R51.1, R52.1, U4.8 (VBUS)
- new net: Q20.2 (B), R49.2
- new net Chip_PU: Q20.1 (C)
- new net DTR: Q21.3 (E), R49.1, U4.28 (~{DTR})
- new net GPIO0: Q21.1 (C)
- new net RTS: Q20.3 (E), R50.1, U4.24 (~{RTS})
- new net U0RXT: U4.26 (TXD)
- new net U0TXD: U4.25 (RXD)
- new net USB_D_N: D5.2 (A2), J12.A7 (D-), J12.B7 (D-), U4.5 (D-)
- new net USB_D_P: D4.2 (A2), J12.A6 (D+), J12.B6 (D+), U4.4 (D+)
- no-connect marks 7 -> 24
Other:
- note added: "USB to UART"
- note added: "USB-C Connector"
