File: Instrument Panel Final.kicad_sch (KiCad schematic)
At the start: 110 parts, among them IC1 LM2678SD-5.0_NOPB, J1 Conn_01x03_Socket, J10 Conn_01x07_Socket, J11 Conn_01x03_Socket, J12 Conn_01x04_Socket, J13 Conn_01x02_Socket, J14 Conn_01x03_Socket, J15 Conn_01x03_Socket, J16 USB_C_Receptacle_USB2.0_14P, J2 Conn_01x07_Socket, J3 Conn_01x07_Socket, J4 Conn_01x03_Socket, J5 Conn_01x06_Socket, J6 Conn_01x03_Socket, J7 Conn_01x05_Socket, J8 Conn_01x03_Socket, J9 Conn_01x03_Socket, Q1 NMOS, Q10 NPN, Q11 NPN, Q2 NMOS, Q3 NMOS, Q4 NMOS, Q5 NMOS, Q6 NMOS, Q7 NMOS, Q8 NMOS, Q9 2N7000, SW1 SW_Push, U1 UA78M33QDCYRQ1, U2 SFH617A-1, U3 ESP32-S3-MINI-1U, U4 24C02Cx-x-SN, U5 24C02Cx-x-SN, U6 CP2102N-Axx-xQFN28, U7 LM7171xIM

Commit message: updated to latest version
Parts:
- removed C1, C2, C3: 15uF, Capacitor_THT:CP_Radial_D5.0mm_P2.50mm, symbol Device:C_Polarized
- removed C10, C14: 1u, Capacitor_THT:C_Disc_D3.0mm_W1.6mm_P2.50mm, symbol Device:C
- removed C11, C13, C16: 10u, Capacitor_THT:C_Disc_D3.0mm_W1.6mm_P2.50mm, symbol Device:C
- removed C12, C15, C6: 0.1u, Capacitor_THT:C_Disc_D3.0mm_W1.6mm_P2.50mm, symbol Device:C
- removed C17: 1000u, Capacitor_THT:CP_Radial_D5.0mm_P2.50mm, symbol Device:C_Polarized
- removed C4: 0.47uF, Capacitor_THT:C_Disc_D3.0mm_W1.6mm_P2.50mm, symbol Device:C
- removed C5: 0.33u, Capacitor_THT:CP_Radial_D5.0mm_P2.50mm, symbol Device:C_Polarized
- removed C7: 0.01uF, Capacitor_THT:C_Disc_D3.0mm_W1.6mm_P2.50mm, symbol Device:C
- removed C8, C9: 180uF, Capacitor_THT:CP_Radial_D5.0mm_P2.50mm, symbol Device:C_Polarized
- removed D1, D14: D_Schottky, Diode_THT:D_A-405_P7.62mm_Horizontal, symbol Device:D_Schottky
- removed D10, D7, D8: SMAJ5.0CA, Diode_SMD:D_SMA, symbol Diode:SMAJ5.0CA
- removed D11: 1N5819, Diode_THT:D_DO-41_SOD81_P10.16mm_Horizontal, symbol Diode:1N5819
- removed D12, D13, D2, D5, D6, D9: APA-106-F5, LED_THT:LED_D5.0mm-4_RGB, symbol LED:APA-106-F5
- removed D15: SMAJ20A, Diode_SMD:D_SMA, symbol Diode:SMAJ20A
- removed D3, D4: D, Diode_THT:D_A-405_P7.62mm_Horizontal, symbol Device:D
- removed F1: AHEF750, Fuse:Fuse_Littelfuse-LVR100, symbol SamacSys_Parts:AHEF750
- removed IC1: LM2678SD-5.0_NOPB, Package_SON:VSON-14-1EP_3x4.45mm_P0.65mm_EP1.6x4.2mm, symbol SamacSys_Parts:LM2678SD-5.0_NOPB
- removed J1, J11, J14, J15, J4, J6, J8, J9: Conn_01x03_Socket, Connector_Molex:Molex_KK-396_A-41791-0003_1x03_P3.96mm_Vertical, symbol Connector:Conn_01x03_Socket
- removed J10, J2, J3: Conn_01x07_Socket, Connector_Molex:Molex_KK-396_5273-07A_1x07_P3.96mm_Vertical, symbol Connector:Conn_01x07_Socket
- removed J12: Conn_01x04_Socket, Connector_Molex:Molex_KK-396_5273-04A_1x04_P3.96mm_Vertical, symbol Connector:Conn_01x04_Socket
- removed J13: Conn_01x02_Socket, Connector_Molex:Molex_KK-254_AE-6410-02A_1x02_P2.54mm_Vertical, symbol Connector:Conn_01x02_Socket
- removed J16: USB_C_Receptacle_USB2.0_14P, Connector_USB:USB_C_Receptacle_GCT_USB4085, symbol Connector:USB_C_Receptacle_USB2.0_14P
- removed J5: Conn_01x06_Socket, Connector_Molex:Molex_KK-396_5273-06A_1x06_P3.96mm_Vertical, symbol Connector:Conn_01x06_Socket
- removed J7: Conn_01x05_Socket, Connector_Molex:Molex_KK-396_5273-05A_1x05_P3.96mm_Vertical, symbol Connector:Conn_01x05_Socket
- removed L1: 22uH, Inductor_THT:L_Radial_D9.5mm_P5.00mm_Fastron_07HVP, symbol Device:L
- removed Q1, Q2, Q3, Q4, Q5, Q6, Q7, Q8: NMOS, Package_TO_SOT_THT:TO-92_Inline, symbol Simulation_SPICE:NMOS
- removed Q10, Q11: NPN, Package_TO_SOT_THT:TO-92_Inline, symbol Simulation_SPICE:NPN
- removed Q9: 2N7000, Package_TO_SOT_THT:TO-92_Inline, symbol Transistor_FET:2N7000
- removed R1, R10, R11, R12, R13, R14, R15, R16, R17, R19, R2, R22, R23, R24, R25, R3, R30, R31, R32, R33, R34, R38, R4, R5, R6, R7, R8, R9: 10K, Resistor_THT:R_Axial_DIN0207_L6.3mm_D2.5mm_P10.16mm_Horizontal, symbol Device:R
- removed R18: 150, Resistor_THT:R_Axial_DIN0207_L6.3mm_D2.5mm_P10.16mm_Horizontal, symbol Device:R
- removed R20, R21, R26, R27, R28, R29: 220, Resistor_THT:R_Axial_DIN0207_L6.3mm_D2.5mm_P10.16mm_Horizontal, symbol Device:R
- removed R35: 22.1K, Resistor_THT:R_Axial_DIN0207_L6.3mm_D2.5mm_P10.16mm_Horizontal, symbol Device:R
- removed R36: 47.5K, Resistor_THT:R_Axial_DIN0207_L6.3mm_D2.5mm_P10.16mm_Horizontal, symbol Device:R
- removed R37: 1K, Resistor_THT:R_Axial_DIN0207_L6.3mm_D2.5mm_P10.16mm_Horizontal, symbol Device:R
- removed R39: 11K, Resistor_THT:R_Axial_DIN0207_L6.3mm_D2.5mm_P10.16mm_Horizontal, symbol Device:R
- removed R40: 10, Resistor_THT:R_Axial_DIN0207_L6.3mm_D2.5mm_P10.16mm_Horizontal, symbol Device:R
- removed SW1: SW_Push, Button_Switch_THT:SW_PUSH_6mm_H8mm, symbol Switch:SW_Push
- removed U1: UA78M33QDCYRQ1, Package_TO_SOT_SMD:SOT-223-3_TabPin2, symbol Regulator_Linear:UA78M33QDCYRQ1
- removed U2: SFH617A-1, Package_DIP:DIP-4_W7.62mm, symbol Isolator:SFH617A-1
- removed U3: ESP32-S3-MINI-1U, RF_Module:ESP32-S2-MINI-1U, symbol RF_Module:ESP32-S3-MINI-1U
- removed U4, U5: 24C02Cx-x-SN, Package_DIP:DIP-8_W7.62mm_Socket, symbol Memory_EEPROM:24C02Cx-x-SN
- removed U6: CP2102N-Axx-xQFN28, Package_DFN_QFN:QFN-28-1EP_5x5mm_P0.5mm_EP3.35x3.35mm, symbol Interface_USB:CP2102N-Axx-xQFN28
- removed U7: LM7171xIM, Package_SO:SOIC-8_3.9x4.9mm_P1.27mm, symbol Amplifier_Operational:LM7171xIM
Connections:
- no-connect marks 27 -> 0
Other:
- added sheet ADC (adc.kicad_sch)
- added sheet Amplifier (amplifier.kicad_sch)
- added sheet Connections (connections.kicad_sch)
- added sheet EEPROM (eeprom.kicad_sch)
- added sheet ESP32 S2 (esp32_s2.kicad_sch)
- added sheet LEDs (leds.kicad_sch)
- added sheet Logic Shifters (logic_shifters.kicad_sch)
- added sheet Power (power.kicad_sch)
- added sheet Push Buttons (push_buttons.kicad_sch)
- added sheet USB (usb.kicad_sch)
- note removed: "Batt LED"
- note removed: "Fuel LED"
- note removed: "Left Turn LED"
- note removed: "Oil LED"
- note removed: "Right Turn LED"
- note removed: "Temp LED"

Commit message: update
Parts:
- added C10: 1u, Capacitor_THT:C_Disc_D3.0mm_W1.6mm_P2.50mm, symbol Device:C
- added C11: 10u, Capacitor_THT:C_Disc_D3.0mm_W1.6mm_P2.50mm, symbol Device:C
- added C12, C19: 0.1u, Capacitor_THT:C_Disc_D3.0mm_W1.6mm_P2.50mm, symbol Device:C
- added C16, C18: 10uF, Capacitor_THT:C_Disc_D3.0mm_W1.6mm_P2.50mm, symbol Device:C
- added C17: 0.1uF, Capacitor_THT:C_Disc_D3.0mm_W1.6mm_P2.50mm, symbol Device:C
- added C20: 1000u, Capacitor_THT:CP_Radial_D5.0mm_P2.50mm, symbol Device:C_Polarized
- added D10, D11, D12, D13, D14, D15, D16, D8, D9: APA-106-F5, LED_THT:LED_D5.0mm-4_RGB, symbol LED:APA-106-F5
- added FB1: FerriteBead_Small, Inductor_THT:L_Axial_L5.0mm_D3.6mm_P10.00mm_Horizontal_Murata_BL01RN1A2A2, symbol Device:FerriteBead_Small
- added J1, J3, J4, J5, J7, J8, J9: Conn_01x03_Socket, Connector_Hirose:Hirose_DF13-03P-1.25DSA_1x03_P1.25mm_Vertical, symbol Connector:Conn_01x03_Socket
- added J10, J11: Conn_01x06_Socket, Connector_Hirose:Hirose_DF13-06P-1.25DSA_1x06_P1.25mm_Vertical, symbol Connector:Conn_01x06_Socket
- added J2: Conn_01x02_Socket, Connector_Hirose:Hirose_DF13-02P-1.25DSA_1x02_P1.25mm_Vertical, symbol Connector:Conn_01x02_Socket
- added J6: Conn_01x23_Socket, Connector_Molex:Molex_SL_171971-0023_1x23_P2.54mm_Vertical, symbol Connector:Conn_01x23_Socket
- added R10, R11, R6, R7, R8, R9: 220, Resistor_THT:R_Axial_DIN0207_L6.3mm_D2.5mm_P10.16mm_Horizontal, symbol Device:R
- added R12, R3, R4, R5: 10k, Resistor_THT:R_Axial_DIN0207_L6.3mm_D2.5mm_P10.16mm_Horizontal, symbol Device:R
- added R2, R55, R56, R57, R58, R59, R60, R62: 10K, Resistor_THT:R_Axial_DIN0207_L6.3mm_D2.5mm_P10.16mm_Horizontal, symbol Device:R
- added R61: 10, Resistor_THT:R_Axial_DIN0207_L6.3mm_D2.5mm_P10.16mm_Horizontal, symbol Device:R
- added SW1, SW2, SW3: SW_Push, Button_Switch_THT:SW_PUSH_6mm_H8mm, symbol Switch:SW_Push
- added U3: ESP32-S2-MINI-2U-N4, ESP32_S2_MINI_2U_N4:XCVR_ESP32-S2-MINI-2U-N4, symbol ESP32-S2-MINI-2U-N4:ESP32-S2-MINI-2U-N4
- added U5: ADS1015IDGS, Package_SO:TSSOP-10_3x3mm_P0.5mm, symbol Analog_ADC:ADS1015IDGS
- added U6, U7: 24C02Cx-x-SN, Package_DIP:DIP-8_W7.62mm, symbol Memory_EEPROM:24C02Cx-x-SN
- added U8: LM7171xIM, Package_DIP:DIP-8_W7.62mm, symbol Amplifier_Operational:LM7171xIM
Connections:
- new net: D11.1 (DO), D13.4 (DI)
- new net: D11.4 (DI), D8.1 (DO)
- new net: D14.1 (DO), D16.4 (DI)
- new net: D12.1 (DO), D14.4 (DI)
- new net: D16.1 (DO), D8.4 (DI)
- new net: C19.1, C20.1, U8.6
- new net: R11.1, U3.19 (IO15)
- new net: R56.2, U6.2 (A1)
- new net: D10.1 (DO), D12.4 (DI)
- new net: R10.1, U3.18 (IO14)
- new net: R9.1, U3.17 (IO13)
- new net: C19.2, R61.1
- new net: R59.2, U7.2 (A1)
- new net: R60.2, U7.3 (A2)
- new net: D10.4 (DI), D9.1 (DO)
- new net: R6.1, U3.14 (IO10)
- new net: R7.1, U3.15 (IO11)
- new net: R8.1, U3.16 (IO12)
- new net: R55.2, U6.1 (A0)
- new net: R57.2, U6.3 (A2)
- new net: D13.1 (DO), D15.4 (DI)
- new net +3.3V: C11.1, C12.1, J10.2 (Pin_2), J11.2 (Pin_2), J6.4 (Pin_4), R12.1, R2.1, R3.1, R4.1, R5.1, R58.2, SW1.1, U3.3 (3V3), U6.8 (VCC), U7.1 (A0), U7.8 (VCC)
- new net +5V: C16.1, D10.3 (VDD), D11.3 (VDD), D12.3 (VDD), D13.3 (VDD), D14.3 (VDD), D15.3 (VDD), D16.3 (VDD), D8.3 (VDD), D9.3 (VDD), FB1.1, J1.3 (Pin_3), J3.2 (Pin_2), J4.2 (Pin_2), J5.2 (Pin_2), J6.7 (Pin_7), J7.2 (Pin_2), J8.2 (Pin_2), J9.2 (Pin_2)
- new net +BATT: J6.9 (Pin_9)
- new net +VDC: J6.10 (Pin_10)
- new net Backlight_Strip: D15.1 (DO), J1.2 (Pin_2)
- new net Batt_In: J6.11 (Pin_11), U5.5 (AIN1)
- new net Batt_Servo: J9.3 (Pin_3), R11.2
- new net Brake_Adjusted: U3.31 (IO35)
- new net Brake_In: J6.22 (Pin_22)
- new net CL: J10.3 (Pin_3), J11.3 (Pin_3), U3.11 (IO7)
- new net CS0: J11.5 (Pin_5), R12.2, U3.9 (IO5)
- new net CS1: J10.5 (Pin_5), R5.2, U3.8 (IO4)
- new net Chip_PU: C10.1, R2.2, SW2.2, U3.45 (EN)
- new net DA: J10.4 (Pin_4), J11.4 (Pin_4), U3.7 (IO3)
- new net DC: J10.6 (Pin_6), J11.6 (Pin_6), U3.6 (IO2)
- new net Echo_Adjusted: U3.34 (IO38)
- new net Echo_In: J6.19 (Pin_19)
- new net Fuel_In: J6.13 (Pin_13), U5.6 (AIN2)
- new net Fuel_Servo: J4.3 (Pin_3), R7.2
- new net GND: C10.2, C11.2, C12.2, C16.2, C17.2, C18.2, D10.2 (GND), D11.2 (GND), D12.2 (GND), D13.2 (GND), D14.2 (GND), D15.2 (GND), D16.2 (GND), D8.2 (GND), D9.2 (GND), J1.1 (Pin_1), J10.1 (Pin_1), J11.1 (Pin_1), J2.1 (Pin_1), J3.1 (Pin_1), J4.1 (Pin_1), J5.1 (Pin_1), J6.1 (Pin_1), J6.5 (Pin_5), J6.8 (Pin_8), J7.1 (Pin_1), J8.1 (Pin_1), J9.1 (Pin_1), R55.1, R56.1, R57.1, R58.1, R59.1, R60.1, R61.2, R62.2, SW2.1, SW3.1, U3.1 (GND1), U3.2 (GND1__1), U3.30 (GND1__2), U3.42 (GND1__3), U3.43 (GND1__4), U3.46 (GND1__5), U3.47 (GND1__6), U3.48 (GND1__7), U3.49 (GND1__8), U3.50 (GND1__9), U3.51 (GND1__10), U3.52 (GND1__11), U3.53 (GND1__12), U3.54 (GND1__13), U3.55 (GND1__14), U3.56 (GND2), U3.57 (GND2__1), U3.58 (GND2__2), U3.59 (GND2__3), U3.60 (GND2__4), U3.61_1 (GND2__5), U3.61_2 (GND2__6), U3.61_3 (GND2__7), U3.61_4 (GND2__8), U3.61_5 (GND2__9), U3.61_6 (GND2__10), U3.61_7 (GND2__11), U3.61_8 (GND2__12), U3.61_9 (GND2__13), U3.62 (GND2__14), U3.63 (GND3), U3.64 (GND3__1), U3.65 (GND3__2), U5.1 (ADDR), U5.3 (GND), U6.4 (GND), U6.7 (WP), U7.4 (GND), U7.7 (WP), U8.2 (-), U8.4 (V-)
- new net GPIO0: SW3.2, U3.4 (IO0)
- new net Hazard_Adjusted: U3.35 (IO39)
- new net Hazard_In: J6.18 (Pin_18)
- new net Headlights_High_Adjusted: U3.29 (IO34)
- new net Headlights_High_In: J6.23 (Pin_23)
- new net Headlights_Low_Adjusted: U3.36 (IO40)
- new net Headlights_Low_In: J6.17 (Pin_17)
- new net Ignition_Sensor: U3.22 (IO18)
- new net LED_Data_Out: D9.4 (DI), U3.5 (IO1)
- new net Left_Turn_Adjusted: U3.33 (IO37)
- new net Left_Turn_In: J6.20 (Pin_20)
- new net Oil_In: J6.14 (Pin_14), U5.7 (AIN3)
- new net Oil_Servo: J3.3 (Pin_3), R6.2
- new net Power_Off: U3.21 (IO17)
- new net Right_Turn_Adjusted: U3.32 (IO36)
- new net Right_Turn_In: J6.21 (Pin_21)
- new net SCL: J6.2 (Pin_2), R3.2, U3.13 (IO9), U5.10 (SCL), U6.6 (SCL), U7.6 (SCL)
- new net SDA: J6.3 (Pin_3), R4.2, U3.12 (IO8), U5.9 (SDA), U6.5 (SDA), U7.5 (SDA)
- new net Sound_out: U3.28 (IO33), U8.3 (+)
- new net Speaker: C20.2, J2.2 (Pin_2)
- new net Speed_Adjusted: U3.37 (IO41)
- new net Speed_In: J6.16 (Pin_16)
- new net Speed_Servo: J5.3 (Pin_3), R8.2
- new net Tach_Adjusted: U3.38 (IO42)
- new net Tach_In: J6.15 (Pin_15)
- new net Tach_Servo: J7.3 (Pin_3), R9.2
- new net Temp_In: J6.12 (Pin_12), U5.4 (AIN0)
- new net Temp_Servo: J8.3 (Pin_3), R10.2
- new net Trigger: J6.6 (Pin_6), U3.20 (IO16)
- new net Trip Reset: R62.1, SW1.2, U3.25 (IO21)
- new net U0RXT: U3.40 (IO44/RXD0)
- new net U0TXD: U3.39 (IO43/TXD0)
- new net VAA: U8.7 (V+)
- new net VDDA: C17.1, C18.1, FB1.2, U5.8 (VDD)
- no-connect marks 0 -> 7
Other:
- removed sheet ADC
- removed sheet Amplifier
- removed sheet Connections
- removed sheet EEPROM
- removed sheet ESP32 S2
- removed sheet LEDs
- removed sheet Power
- removed sheet Push Buttons
- removed sheet USB
- added sheet USB and Power (power.kicad_sch)
- note added: "ADC"
- note added: "Addr 0x48"
- note added: "Amplifier"
- note added: "Batt LED"
- note added: "Brake LED"
- note added: "EEPROMs"
- note added: "External Connector"
- note added: "Fuel LED"
- note added: "High Beam LED"
- note added: "Internal Connectors"
- note added: "LEDs"
- note added: "Left Turn LED"
- note added: "Low Beam LED"
- note added: "Oil LED"
- note added: "Right Turn LED"
- note added: "Temp LED"

Commit message: update
Parts:
- added U10, U11, U9: 74HC595, Package_DIP:DIP-16_W7.62mm, symbol 74xx:74HC595
- added U12, U13, U14, U15, U16, U17: L293D, Package_DIP:DIP-16_W7.62mm, symbol Driver_Motor:L293D
