File: Instrument Panel Final.kicad_sch (KiCad schematic)
At the start: 65 parts, among them J1 Conn_01x03_Socket, J10 Conn_01x06_Socket, J11 Conn_01x06_Socket, J2 Conn_01x02_Socket, J3 Conn_01x03_Socket, J4 Conn_01x03_Socket, J5 Conn_01x03_Socket, J6 Conn_01x23_Socket, J7 Conn_01x03_Socket, J8 Conn_01x03_Socket, J9 Conn_01x03_Socket, SW1 SW_Push, SW2 SW_Push, SW3 SW_Push, U10 74HC595, U11 74HC595, U12 L293D, U13 L293D, U14 L293D, U15 L293D, U16 L293D, U17 L293D, U3 ESP32-S2-MINI-2U-N4, U5 ADS1015IDGS, U6 24C02Cx-x-SN, U7 24C02Cx-x-SN, U8 LM7171xIM, U9 74HC595

Commit message: update
Parts:
- removed J3, J4, J5, J7, J8, J9: Conn_01x03_Socket, Connector_Hirose:Hirose_DF13-03P-1.25DSA_1x03_P1.25mm_Vertical, symbol Connector:Conn_01x03_Socket
- removed R10, R11, R6, R7, R8, R9: 220, Resistor_THT:R_Axial_DIN0207_L6.3mm_D2.5mm_P10.16mm_Horizontal, symbol Device:R
- removed U10, U11, U9: 74HC595, Package_DIP:DIP-16_W7.62mm, symbol 74xx:74HC595
- removed U12, U13, U14, U15, U16, U17: L293D, Package_DIP:DIP-16_W7.62mm, symbol Driver_Motor:L293D
- added R66: 10k, Resistor_THT:R_Axial_DIN0207_L6.3mm_D2.5mm_P10.16mm_Horizontal, symbol Device:R
Connections:
- net +3.3V: now also R66.1
- net CS2: now reaches U3.19 (IO15)
- net CS2: now also R66.2
- no-connect marks 7 -> 12
Other:
- added sheet Motor Drivers and Shift Registers (motor_drivers_shift_registers.kicad_sch)
